File: project1/LattepndaCourse/LaPandaModule.kicad_sch (KiCad schematic)
At the start: 0 parts

Commit message: Hierachi
Parts:
- added A1: LattePanda_Mu, Module_LattePanda:LattePanda_Module_H8.0mm_Horizontal, symbol MCU_Module_LattePanda:LattePanda_Mu
Connections:
- new net: A1.101 (GND), A1.107 (GND), A1.11 (GND), A1.110 (GND), A1.113 (GND), A1.116 (GND), A1.135 (GND), A1.136 (GND), A1.14 (GND), A1.151 (GND), A1.158 (GND), A1.167 (GND), A1.17 (GND), A1.170 (GND), A1.181 (GND), A1.182 (GND), A1.188 (GND), A1.189 (GND), A1.194 (GND), A1.195 (GND), A1.20 (GND), A1.200 (GND), A1.201 (GND), A1.206 (GND), A1.207 (GND), A1.212 (GND), A1.213 (GND), A1.218 (GND), A1.219 (GND), A1.224 (GND), A1.225 (GND), A1.23 (GND), A1.230 (GND), A1.231 (GND), A1.236 (GND), A1.237 (GND), A1.242 (GND), A1.243 (GND), A1.248 (GND), A1.249 (GND), A1.26 (GND), A1.29 (GND), A1.32 (GND), A1.35 (GND), A1.38 (GND), A1.41 (GND), A1.44 (GND), A1.47 (GND), A1.50 (GND), A1.53 (GND), A1.56 (GND), A1.59 (GND), A1.62 (GND), A1.65 (GND), A1.68 (GND), A1.71 (GND), A1.74 (GND), A1.77 (GND), A1.80 (GND), A1.83 (GND), A1.86 (GND), A1.89 (GND), A1.92 (GND), A1.95 (GND), A1.98 (GND)
- new net: A1.250 (VIN), A1.251 (VIN), A1.252 (VIN), A1.253 (VIN), A1.254 (VIN), A1.255 (VIN), A1.256 (VIN), A1.257 (VIN), A1.258 (VIN), A1.259 (VIN), A1.260 (VIN)
Other:
- title: (none) -> practice design
