File: project1/LattepndaCourse/LaPandaModule.kicad_sch (KiCad schematic)
At the start: 1 part

Commit message: test2
Other:
- note added: "Testing github"
Changed lines of the file:
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@@
 (kicad_sch
-	(version 20250114)
+	(version 20260306)
 	(generator "eeschema")
-	(generator_version "9.0")
+	(generator_version "10.0")
 	(paper "A2")
 	(title_block
@@
 		(rev "1")
 	)
+	(text "Testing github"
+		(exclude_from_sim no)
+		(at 226.06 181.102 0)
+		(effects
+			(font
+				(size 5.08 5.08)
+				(thickness 1.016)
+				(bold yes)
+				(color 255 51 215 1)
+			)
+		)
+	)
 	(no_connect
 		(at 255.27 195.58)
@@
 		(at 295.91 195.58 0)
 		(unit 1)
+		(body_style 1)
 		(exclude_from_sim no)
 		(in_bom yes)
 		(on_board yes)
+		(in_pos_files yes)
 		(dnp no)
 		(fields_autoplaced yes)
 		(property "Reference" "A1"
 			(at 300.5933 58.42 0)
+			(show_name no)
+			(do_not_autoplace no)
 			(effects
 				(font
@@
 		(property "Value" "LattePanda_Mu"
 			(at 300.5933 60.96 0)
+			(show_name no)
+			(do_not_autoplace no)
 			(effects
 				(font
@@
 		(property "Footprint" "Module_LattePanda:LattePanda_Module_H8.0mm_Horizontal"
 			(at 295.91 185.42 0)
+			(hide yes)
+			(show_name no)
+			(do_not_autoplace no)
 			(effects
 				(font
 					(size 1.27 1.27)
 				)
-				(hide yes)
 			)
 		)
 		(property "Datasheet" ""
 			(at 295.91 185.42 0)
+			(hide yes)
+			(show_name no)
+			(do_not_autoplace no)
 			(effects
 				(font
 					(size 1.27 1.27)
 				)
-				(hide yes)
 			)
 		)
 		(property "Description" "A micro computing module with x86 processer, RAM and eMMC."
 			(at 295.91 195.58 0)
+			(hide yes)
+			(show_name no)
+			(do_not_autoplace no)
 			(effects
 				(font
 					(size 1.27 1.27)
 				)
-				(hide yes)
 			)
 		)
@@
 		)
 		(instances
-			(project ""
+			(project "LattepndaCourse"
 				(path "/4e04f3a7-ba43-4db9-8bbc-1a27efcf5abf/e658b8ed-bbad-487b-848e-8e04e48b43c0"
 					(reference "A1")

Commit message: 9/30/36 10pm
Parts:
- added BT1: Battery_Cell, symbol Device:Battery_Cell
- added R1, R2, R3: 10K/1%, symbol Device:R
- added R4, R5: 100K/1%, symbol Device:R
- added R6: 1K/1%, symbol Device:R
- added TP1: TestPoint, symbol Connector:TestPoint
Connections:
- net at A1.100 (~{CLKREQ3}): now also R3.2
- net GND: now reaches A1.101 (GND), A1.107 (GND), A1.11 (GND), A1.110 (GND), A1.113 (GND), A1.116 (GND), A1.135 (GND), A1.136 (GND), A1.14 (GND), A1.151 (GND), A1.158 (GND), A1.167 (GND), A1.17 (GND), A1.170 (GND), A1.181 (GND), A1.182 (GND), A1.188 (GND), A1.189 (GND), A1.194 (GND), A1.195 (GND), A1.20 (GND), A1.200 (GND), A1.201 (GND), A1.206 (GND), A1.207 (GND), A1.212 (GND), A1.213 (GND), A1.218 (GND), A1.219 (GND), A1.224 (GND), A1.225 (GND), A1.23 (GND), A1.230 (GND), A1.231 (GND), A1.236 (GND), A1.237 (GND), A1.242 (GND), A1.243 (GND), A1.248 (GND), A1.249 (GND), A1.26 (GND), A1.29 (GND), A1.32 (GND), A1.35 (GND), A1.38 (GND), A1.41 (GND), A1.44 (GND), A1.47 (GND), A1.50 (GND), A1.53 (GND), A1.56 (GND), A1.59 (GND), A1.62 (GND), A1.65 (GND), A1.68 (GND), A1.71 (GND), A1.74 (GND), A1.77 (GND), A1.80 (GND), A1.83 (GND), A1.86 (GND), A1.89 (GND), A1.92 (GND), A1.95 (GND), A1.98 (GND)
- net GND: now also A1.MP (Mountinge_Pads), BT1.2 (-), R2.1, R3.1, R4.2, R5.2
- net at A1.102 (~{CLKREQ4}): now also R2.2
- net +BATT: now reaches A1.115 (VBAT)
- net +BATT: now also R6.2
- net at A1.133 (~{BIOS_SEL}): now also R1.1, TP1.1
- net at A1.185 (TCP1_HPD): now also R5.1
- net at A1.187 (TCP0_HPD): now also R4.1
- net VDC: now reaches A1.250 (VIN), A1.251 (VIN), A1.252 (VIN), A1.253 (VIN), A1.254 (VIN), A1.255 (VIN), A1.256 (VIN), A1.257 (VIN), A1.258 (VIN), A1.259 (VIN), A1.260 (VIN)
- new net: BT1.1 (+), R6.1
- new net PullUp: R1.2
Other:
- note removed: "Testing github"

Commit message: continue
Parts:
- added J1: Conn_01x03_Pin, A_HDJ_Library:PinHeader_1x03_P2.54mm_Vertical, symbol Connector:Conn_01x03_Pin
Connections:
- net GND: now also J1.3 (Pin_3)
- net ~{PWR_SW}: now reaches A1.1 (~{PWRBTN})
- net at A1.10 (SIO_UART_TX): now also J1.1 (Pin_1)
- net at A1.12 (SIO_UART_RX): now also J1.2 (Pin_2)
- net ~{RST_SW}: now reaches A1.3 (~{RSTBTN})
- net ~{PWR_LED}: now reaches A1.5 (SLS_S0)

Commit message: A
Connections:
- net HSIO_0_TX+: now reaches A1.13 (HSIO0_TX+)
- net HSIO_0_TX-: now reaches A1.15 (HSIO0_TX-)
- net HSIO_0_RX+: now reaches A1.16 (HSIO0_RX+)
- net HSIO_0_RX-: now reaches A1.18 (HSIO0_RX-)
- net HSIO_1_TX+: now reaches A1.19 (HSIO1_TX+)
- net HSIO_1_TX-: now reaches A1.21 (HSIO1_TX-)
- net HSIO_1_RX+: now reaches A1.22 (HSIO1_RX+)
- net HSIO_1_RX-: now reaches A1.24 (HSIO1_RX-)
- net HSIO_2_TX+: now reaches A1.25 (HSIO2_TX+)
- net HSIO_2_TX-: now reaches A1.27 (HSIO2_TX-)
- net HSIO_2_RX+: now reaches A1.28 (HSIO2_RX+)
- net HSIO_2_RX-: now reaches A1.30 (HSIO2_RX-)
- net HSIO_3_TX+: now reaches A1.31 (HSIO3_TX+)
- net HSIO_3_TX-: now reaches A1.33 (HSIO3_TX-)
- net HSIO_3_RX+: now reaches A1.34 (HSIO3_RX+)
- net HSIO_3_RX-: now reaches A1.36 (HSIO3_RX-)
- net HSIO_8_TX+: now reaches A1.37 (HSIO8_TX+)
- net HSIO_8_TX-: now reaches A1.39 (HSIO8_TX-)
- net HSIO_8_RX+: now reaches A1.40 (HSIO8_RX+)
- net HSIO_8_RX-: now reaches A1.42 (HSIO8_RX-)
- net HSIO_9_TX+: now reaches A1.43 (HSIO9_TX+)
- net HSIO_9_TX-: now reaches A1.45 (HSIO9_TX-)
- net HSIO_9_RX+: now reaches A1.46 (HSIO9_RX+)
- net HSIO_9_RX-: now reaches A1.48 (HSIO9_RX-)
- net HSIO_10_TX+: now reaches A1.49 (HSIO10_TX+)
- net HSIO_10_TX-: now reaches A1.51 (HSIO10_TX-)
- net HSIO_10_RX+: now reaches A1.52 (HSIO10_RX+)
- net HSIO_10_RX-: now reaches A1.54 (HSIO10_RX-)
- net HSIO_11_TX+: now reaches A1.55 (HSIO11_TX+)
- net HSIO_11_TX-: now reaches A1.57 (HSIO11_TX-)
- net HSIO_11_RX+: now reaches A1.58 (HSIO11_RX+)
- net HSIO_11_RX-: now reaches A1.60 (HSIO11_RX-)
- net SLS_S3: now reaches A1.7 (SLS_S3)
- net ~{PWR_LED} renamed ~{PWR_LED}/~{PSON}

Commit message: LattePand sheet is done
Connections:
- net ~{WAKE}: now reaches A1.103 (~{WAKE})
- net ~{PLTRST}: now reaches A1.105 (~{PLTRST})
- net USB2_P5-: now reaches A1.109 (USB2_P5-)
- net USB2_P5+: now reaches A1.111 (USB2_P5+)
- net GPP_D0: now reaches A1.128 (GPP_D0)
- net GPP_D1: now reaches A1.130 (GPP_D1)
- net SUSCLK_WIFI: now reaches A1.131 (SUSCLK)
- net GPP_D2: now reaches A1.132 (GPP_D2)
- net GPP_D3: now reaches A1.134 (GPP_D3)
- net UART0_RXD: now reaches A1.137 (UART0_RXD)
- net UART2_TXD: now reaches A1.138 (UART2_TXD)
- net UART0_TXD: now reaches A1.139 (UART0_TXD)
- net UART2_RXD: now reaches A1.140 (UART2_RXD)
- net UART1_RXD: now reaches A1.141 (UART1_RXD)
- net I2C5_SCL: now reaches A1.142 (I2C5_SCL)
- net UART1_TXD: now reaches A1.143 (UART1_TXD)
- net I2C5_SDA: now reaches A1.144 (I2C5_SDA)
- net I2C4_SCL: now reaches A1.146 (I2C4_SCL)
- net I2C4_SDA: now reaches A1.148 (I2C4_SDA)
- net I2C3_SCL: now reaches A1.150 (I2C3_SCL)
- net I2C3_SDA: now reaches A1.152 (I2C3_SDA)
- net I2C2_SCL: now reaches A1.154 (I2C2_SCL)
- net I2C2_SDA: now reaches A1.156 (I2C2_SDA)
- net DDIB_DDC_SDA: now reaches A1.169 (DDIB_DDC_SDA)
- net DDIB_DDC_SCL: now reaches A1.171 (DDIB_DDC_SCL)
- net DDIB_HPD: now reaches A1.183 (DDIB_HPD)
- net DDIB_TX3-: now reaches A1.197 (DDIB_TX3-)
- net DDIB_TX3+: now reaches A1.199 (DDIB_TX3+)
- net FAN1_PWM: now reaches A1.2 (FAN1_PWM)
- net DDIB_TX2-: now reaches A1.203 (DDIB_TX2-)
- net DDIB_TX2+: now reaches A1.205 (DDIB_TX2+)
- net DDIB_TX1-: now reaches A1.209 (DDIB_TX1-)
- net DDIB_TX1+: now reaches A1.211 (DDIB_TX1+)
- net DDIB_TX0-: now reaches A1.215 (DDIB_TX0-)
- net DDIB_TX0+: now reaches A1.217 (DDIB_TX0+)
- net FAN1_TAC: now reaches A1.4 (FAN1_TAC)
- net HSIO_6_TX+: now reaches A1.61 (HSIO6_TX+)
- net HSIO_6_TX-: now reaches A1.63 (HSIO6_TX-)
- net HSIO_6_RX+: now reaches A1.64 (HSIO6_RX+)
- net HSIO_6_RX-: now reaches A1.66 (HSIO6_RX-)
- net USB2_P1-: now reaches A1.67 (USB2_P1-)
- net USB2_P1+: now reaches A1.69 (USB2_P1+)
- net USB2_P4+: now reaches A1.70 (USB2_P4+)
- net USB2_P4-: now reaches A1.72 (USB2_P4-)
- net USB2_P2-: now reaches A1.73 (USB2_P2-)
- net USB2_P2+: now reaches A1.75 (USB2_P2+)
- net USB2_P7+: now reaches A1.76 (USB2_P7+)
- net USB2_P7-: now reaches A1.78 (USB2_P7-)
- net USB2_P3-: now reaches A1.79 (USB2_P3-)
- net USB2_P3+: now reaches A1.81 (USB2_P3+)
- net USB2_P8+: now reaches A1.82 (USB2_P8+)
- net USB2_P8-: now reaches A1.84 (USB2_P8-)
- net REFCLK0+: now reaches A1.85 (REFCLK0+)
- net REFCLK0-: now reaches A1.87 (REFCLK0-)
- net REFCLK3+: now reaches A1.88 (REFCLK3+)
- net REFCLK3-: now reaches A1.90 (REFCLK3-)
- net REFCLK4+: now reaches A1.94 (REFCLK4+)
- net REFCLK4-: now reaches A1.96 (REFCLK4-)
- net REFCLK2+: now reaches A1.97 (REFCLK2+)
- net REFCLK2-: now reaches A1.99 (REFCLK2-)
- net SLS_S3: no longer names the net of A1.7 (SLS_S3)
- net ~{PWR_LED}/~{PSON}: no longer names the net of A1.5 (SLS_S0)
- net ~{PWR_SW}: no longer names the net of A1.1 (~{PWRBTN})
- net ~{RST_SW}: no longer names the net of A1.3 (~{RSTBTN})
- no-connect marks 87 -> 80
Other:
- note added: "All I2C have integrated pull-up resistors. No need to add pull-up resistors"
- note added: "Before starting design, you should choose one of the available BIOS configuration on: https://github.com/LattePandaTeam/LattePanda-Mu or contact technical support for custom your BIOS"
- note added: "Before starting design, you should choose one of the available BIOS configuration on: https://github.com/LattePandaTeam/LattePanda-Mu or contact technical support for custom your BIOS The defualt funtions are defined as follows: -DDIA: eDP 1.4b (the 40 pin connector on Mu) -DDIB: HDMI 2.0 -TCP0: HDMI 2.0 -TCP1: USB TypeC (needed external PD controller)"
- note added: "DDI B used for HDMI"
- note added: "HPD pin of unused DDI/TCP port needs to be pulled down"
- note added: "HSIO functions are defined by the BIOS source code connot be changed in BIOS settings"
- note added: "HSIO_0/HSIO_1 used for USB3.0"
- note added: "HSIO_2 used for M.2 M KEY"
- note added: "HSIO_3 used for M.2 E KEY"
- note added: "HSIO_6 used for GbE(PCIe x1)"
- note added: "HSIO_8/9/10/11 used for PCIe x4"
- note added: "Lite Carrier has no second BIOS ROM ~{BIOS_SEL} pull up to 3.3V to select ROM on LattePanda Mu"
- note added: "SPI is only used to connect to the BIOS and discrete TPM. Cannot be used as a general SPI interface."
- note added: "Sleeping State Signal -SLS_SO: -S0 (Working): HIGH -S3 (Sleeping): LOW -S4 (Hibernation): LOW -S3 (Soft Off): LOW -SLS_SO: -S0 (Working): HIGH -S3 (Sleeping): LOW -S4 (Hibernation): LOW -S3 (Soft Off): LOW"
- note added: "The default funtions ared defined as follows: -HSIO0: USB3.2 10Gbps -HSIO1: USB3.2 10Gbps -HSIO2: PCIe 3.0 x1 -HSIO3: PCIe 3.0 x1 -HSIO8: PCIe 3.0 x4 (lane 0) -HSIO9: PCIe 3.0 x4 (lane 1) -HSIO10: PCIe 3.0 x4 (lane 2) -HSIO11: PCIe 3.0 x4 (lane 3) -HSIO6: PCIe 3.0 x1"
- note added: "USB2 P1/P2 used for USB3.0"
- note added: "USB2 P3/P4 used for USB2.0"
- note added: "USB2_P6 is reserved for TypeC PD controller Do not use it as a normal USB"
- note added: "~{CLKREQ} is reserved for PCIe ASPM L1s Unless the device clearly support it, pull it down to enhance compatiblity"

Commit message: power is done
Connections:
- net ~{PWR_SW}: now reaches A1.1 (~{PWRBTN})
- net ~{RST_SW}: now reaches A1.3 (~{RSTBTN})
- net ~{PWR_LED}/~{PSON}: now reaches A1.5 (SLS_S0)
- net SLS_S3: now reaches A1.7 (SLS_S3)
Changed lines of the file:
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@@
 	(wire
 		(pts
+			(xy 250.19 71.12) (xy 255.27 71.12)
+		)
+		(stroke
+			(width 0)
+			(type default)
+		)
+	)
+	(wire
+		(pts
 			(xy 336.55 177.8) (xy 340.36 177.8)
 		)
@@
 	(wire
 		(pts
+			(xy 250.19 68.58) (xy 255.27 68.58)
+		)
+		(stroke
+			(width 0)
+			(type default)
+		)
+	)
+	(wire
+		(pts
 			(xy 250.19 241.3) (xy 255.27 241.3)
 		)
@@
 	(wire
 		(pts
+			(xy 250.19 66.04) (xy 255.27 66.04)
+		)
+		(stroke
+			(width 0)
+			(type default)
+		)
+	)
+	(wire
+		(pts
 			(xy 205.74 78.74) (xy 255.27 78.74)
 		)
@@
 	(wire
 		(pts
+			(xy 250.19 73.66) (xy 255.27 73.66)
+		)
+		(stroke
+			(width 0)
+			(type default)
+		)
+	)
+	(wire
+		(pts
 			(xy 336.55 105.41) (xy 340.36 105.41)
 		)
@@
 		)
 	)
+	(global_label "~{PWR_LED}{slash}~{PSON}"
+		(shape output)
+		(at 250.19 71.12 180)
+		(fields_autoplaced yes)
+		(effects
+			(font
+				(size 1.27 1.27)
+			)
+			(justify right)
+		)
+		(property "Intersheetrefs" "${INTERSHEET_REFS}"
+			(at 232.3277 71.12 0)
+			(hide yes)
+			(show_name no)
+			(do_not_autoplace no)
+			(effects
+				(font
+					(size 1.27 1.27)
+				)
+				(justify right)
+			)
+		)
+	)
 	(global_label "REFCLK4-"
 		(shape output)
@@
 		)
 	)
+	(global_label "~{PWR_SW}"
+		(shape input)
+		(at 250.19 66.04 180)
+		(fields_autoplaced yes)
+		(effects
+			(font
+				(size 1.27 1.27)
+			)
+			(justify right)
+		)
+		(property "Intersheetrefs" "${INTERSHEET_REFS}"
+			(at 239.5849 66.04 0)
+			(hide yes)
+			(show_name no)
+			(do_not_autoplace no)
+			(effects
+				(font
+					(size 1.27 1.27)
+				)
+				(justify right)
+			)
+		)
+	)
 	(global_label "HSIO_1_TX-"
 		(shape output)
@@
 		)
 	)
+	(global_label "~{RST_SW}"
+		(shape input)
+		(at 250.19 68.58 180)
+		(fields_autoplaced yes)
+		(effects
+			(font
+				(size 1.27 1.27)
+			)
+			(justify right)
+		)
+		(property "Intersheetrefs" "${INTERSHEET_REFS}"
+			(at 240.1292 68.58 0)
+			(hide yes)
+			(show_name no)
+			(do_not_autoplace no)
+			(effects
+				(font
+					(size 1.27 1.27)
+				)
+				(justify right)
+			)
+		)
+	)
 	(global_label "UART1_RXD"
 		(shape input)
@@
 			)
 		)
+	)
+	(global_label "SLS_S3"
+		(shape output)
+		(at 250.19 73.66 180)
+		(fields_autoplaced yes)
+		(effects
+			(font
+				(size 1.27 1.27)
+			)
+			(justify right)
+		)
+		(property "Intersheetrefs" "${INTERSHEET_REFS}"
+			(at 240.3711 73.66 0)
+			(hide yes)
+			(show_name no)
+			(do_not_autoplace no)
+			(effects
+				(font
+					(size 1.27 1.27)
+				)
+				(justify right)
+			)
+		)

Commit message: Hierachi needs some work
Connections:
- net FAN2_PWM: now reaches A1.6 (FAN2_PWM)
- net FAN2_TAC: now reaches A1.8 (FAN2_TAC)
- net TSENSE: now reaches A1.9 (TSENSE)
- net DDIB_DDC_SCL renamed DDI_B_DDC_SCL
- net DDIB_DDC_SDA renamed DDI_B_DDC_SDA
- net DDIB_HPD renamed DDI_B_HPD
- net DDIB_TX0+ renamed DDI_B_TX0+
- net DDIB_TX0- renamed DDI_B_TX0-
- net DDIB_TX1+ renamed DDI_B_TX1+
- net DDIB_TX1- renamed DDI_B_TX1-
- net DDIB_TX2+ renamed DDI_B_TX2+
- net DDIB_TX2- renamed DDI_B_TX2-
- net DDIB_TX3+ renamed DDI_B_TX3+
- net DDIB_TX3- renamed DDI_B_TX3-
- no-connect marks 80 -> 77

Commit message: fixing Hierachi
Connections:
- net UART0_RXD renamed SCO_UART0_RX
- net UART0_TXD renamed SCO_UART0_TX
- net UART1_RXD renamed SCO_UART1_RX
- net UART1_TXD renamed SCO_UART1_TX
- net UART2_RXD renamed SCO_UART2_RX
- net UART2_TXD renamed SCO_UART2_TX
Changed lines of the file:
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@@
 		)
 	)
-	(hierarchical_label "UART2_TXD"
+	(hierarchical_label "SCO_UART2_TX"
 		(shape output)
 		(at 340.36 195.58 0)
@@
 		)
 	)
-	(hierarchical_label "UART0_RXD"
+	(hierarchical_label "SCO_UART0_RX"
 		(shape input)
 		(at 340.36 182.88 0)
@@
 		)
 	)
-	(hierarchical_label "UART2_RXD"
+	(hierarchical_label "SCO_UART2_RX"
 		(shape input)
 		(at 340.36 193.04 0)
@@
 		)
 	)
-	(hierarchical_label "UART1_RXD"
+	(hierarchical_label "SCO_UART1_RX"
 		(shape input)
 		(at 340.36 187.96 0)
@@
 		)
 	)
-	(hierarchical_label "UART1_TXD"
+	(hierarchical_label "SCO_UART1_TX"
 		(shape output)
 		(at 340.36 190.5 0)
@@
 		)
 	)
-	(hierarchical_label "UART0_TXD"
+	(hierarchical_label "SCO_UART0_TX"
 		(shape output)
 		(at 340.36 185.42 0)
