File: project1/LattepndaCourse/LaPandaModule.kicad_sch (KiCad schematic)
At the start: 10 parts, among them J1 Conn_01x03_Pin

Commit message: Started routing
Parts:
- added H7, H8: MountingHole_Pad, A_HDJ_Library:MountingHole_3mm_M2_Pad_TopOnly, symbol Mechanical:MountingHole_Pad
- BT1: footprint (none) -> A_HDJ_Library:Battery_Holder_CR1220_S8411-45R
- R1, R2, R3, R4, R5, R6: footprint (none) -> A_HDJ_Library:R_0402_1005Metric
- TP1: footprint (none) -> A_HDJ_Library:TestPoint_Pad_D1.5mm
Connections:
- net GND: now also H7.1, H8.1
