File: project1/LattepndaCourse/M2MKey.kicad_sch (KiCad schematic)
At the start: 0 parts

Commit message: Hierachi
Other:
- title: (none) -> practice design
Changed lines of the file:
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@@
 	(generator "eeschema")
 	(generator_version "9.0")
-	(paper "A4")
+	(paper "A2")
+	(title_block
+		(title "practice design")
+		(date "2026-09-30")
+		(rev "1")
+	)
 )

Commit message: Hierachi needs some work
Parts:
- added C72, C74, C79, C81: 100nF/50V, A_HDJ_Library:C_0603_1608Metric, symbol Device:C_Small
- added C73, C75, C78, C80: 10uF/50V, A_HDJ_Library:C_0603_1608Metric, symbol Device:C_Small
- added C76, C77, C82, C83: 220nF/50V, A_HDJ_Library:C_0603_1608Metric, symbol Device:C_Small
- added D27: LED_G, A_HDJ_Library:LED_0603_1608Metric, symbol Device:LED
- added H5, H6: MountingHole_Pad, symbol Mechanical:MountingHole_Pad
- added J20: Bus_M.2_Socket_M, A_HDJ_Library:PCIe_M.2_Connectors_P=0.5mm_H=4.2mm_KeyM, symbol Connector:Bus_M.2_Socket_M
- added J21: Bus_M.2_Socket_E, A_HDJ_Library:PCIe_M.2_Connectors_P=0.5mm_H=4.2mm_KeyE, symbol Connector:Bus_M.2_Socket_E
- added R65, R68, R69, R70, R71: 0R/1%, A_HDJ_Library:R_0402_1005Metric, symbol Device:R
- added R72, R73: 10K/1%, A_HDJ_Library:R_0402_1005Metric, symbol Device:R
- added TP14: TestPoint, symbol Connector:TestPoint
Connections:
- new net: J21.50 (SUSCLK), R71.1
- new net: J21.54 (~{W_DISABLE2}), R72.1
- new net: J21.56 (~{W_DISABLE1}), R73.1
- new net: D27.1 (K), J20.10 (DAS/~{DSS}/~{LED1})
- new net: J20.38 (DEVSLP), TP14.1
- new net: J20.68 (SUSCLK), R68.1
- new net: J20.69 (PEDET), R69.1
- new net +3V3: C72.1, C73.2, C74.2, C75.2, C78.2, C79.2, C80.2, C81.1, D27.2 (A), J20.12 (3.3V), J20.14 (3.3V), J20.16 (3.3V), J20.18 (3.3V), J20.2 (3.3V), J20.4 (3.3V), J20.70 (3.3V), J20.72 (3.3V), J20.74 (3.3V), J21.2 (3.3V), J21.4 (3.3V), J21.72 (3.3V), J21.74 (3.3V), R72.2, R73.2
- new net CON_PCIE_TX1+: C76.1, C82.1, J20.49 (PETp0/SATA-A+), J21.35 (PETp0)
- new net CON_PCIE_TX1-: C77.1, C83.1, J20.47 (PETn0/SATA-A-), J21.37 (PETn0)
- new net GND: C72.2, C73.1, C74.1, C75.1, C78.1, C79.1, C80.1, C81.2, H5.1, H6.1, J20.1 (GND), J20.15 (GND), J20.21 (GND), J20.27 (GND), J20.3 (GND), J20.33 (GND), J20.39 (GND), J20.45 (GND), J20.51 (GND), J20.57 (GND), J20.71 (GND), J20.73 (GND), J20.75 (GND), J20.9 (GND), J21.1 (GND), J21.18 (GND), J21.33 (GND), J21.39 (GND), J21.45 (GND), J21.51 (GND), J21.57 (GND), J21.63 (GND), J21.69 (GND), J21.7 (GND), J21.75 (GND), R65.1, R69.2, R70.1
- new net PCIE_RX_0+: J21.41 (PERp0)
- new net PCIE_RX_0-: J21.43 (PERn0)
- new net PCIE_RX_1+: J20.43 (PERp0/SATA-B-)
- new net PCIE_RX_1-: J20.41 (PERn0/SATA-B+)
- new net PCIE_TX_0+: C82.2
- new net PCIE_TX_0-: C83.2
- new net PCIE_TX_1+: C76.2
- new net PCIE_TX_1-: C77.2
- new net REFCLKM+: J20.55 (REFCLKp)
- new net REFCLKM-: J20.53 (REFCLKn)
- new net SUSCLK: R68.2, R71.2
- new net USB_2_P7+: J21.3 (USB_D+), J21.47 (REFCLKp0)
- new net USB_2_P7-: J21.49 (REFCLKn0), J21.5 (USB_D-)
- new net ~{CLKREQE}: J21.53 (~{CLKREQ0}), R70.2
- new net ~{CLKREQM}: J20.52 (~{CLKREQ}), R65.2
- new net ~{PLT_RST}: J20.50 (~{PERST}), J21.52 (~{PERST0})
- new net ~{WAKE}: J20.54 (~{PEWAKE}), J21.55 (~{PEWAKE0})
- no-connect marks 0 -> 50

Commit message: fixing Hierachi
Connections:
- net USB_2_P7+: no longer J21.47 (REFCLKp0)
- net USB_2_P7-: no longer J21.49 (REFCLKn0)
- new net REFCLKE+: J21.47 (REFCLKp0)
- new net REFCLKE-: J21.49 (REFCLKn0)
