File: project1/LattepndaCourse/M2MKey.kicad_sch (KiCad schematic)
At the start: 25 parts, among them J20 Bus_M.2_Socket_M, J21 Bus_M.2_Socket_E

Commit message: Started routing
Parts:
- H5, H6: footprint (none) -> A_HDJ_Library:MountingHole_3.2mm_M3_Pad_Via
- TP14: footprint (none) -> A_HDJ_Library:TestPoint_Pad_D1.5mm
