File: project1/LattepndaCourse/LattepndaCourse.kicad_sch (KiCad schematic)
At the start: 6 parts

Commit message: Hierachi
Changed lines of the file:
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@@
 	)
 	(sheet
-		(at 185.42 233.68)
-		(size 12.7 44.45)
+		(at 328.93 143.51)
+		(size 43.18 49.53)
 		(exclude_from_sim no)
 		(in_bom yes)
@@
 		)
 		(property "Sheetname" "GPIO"
-			(at 185.42 232.9684 0)
+			(at 328.93 142.7984 0)
 			(effects
 				(font
@@
 		)
 		(property "Sheetfile" "GPIO.kicad_sch"
-			(at 185.42 278.7146 0)
+			(at 328.93 193.6246 0)
 			(effects
 				(font
@@
 	)
 	(sheet
-		(at 215.9 245.11)
-		(size 12.7 29.21)
+		(at 194.31 68.58)
+		(size 45.72 29.21)
 		(exclude_from_sim no)
 		(in_bom yes)
@@
 		)
 		(property "Sheetname" "Fan"
-			(at 215.9 244.3984 0)
+			(at 194.31 67.8684 0)
 			(effects
 				(font
@@
 		)
 		(property "Sheetfile" "Fan.kicad_sch"
-			(at 215.9 274.9046 0)
+			(at 194.31 98.3746 0)
 			(effects
 				(font
@@
 	)
 	(sheet
-		(at 337.82 229.87)
-		(size 12.7 39.37)
+		(at 328.93 88.9)
+		(size 43.18 46.99)
 		(exclude_from_sim no)
 		(in_bom yes)
@@
 		)
 		(property "Sheetname" "HDMI"
-			(at 337.82 229.1584 0)
+			(at 328.93 88.1884 0)
 			(effects
 				(font
@@
 		)
 		(property "Sheetfile" "HDMI.kicad_sch"
-			(at 337.82 269.8246 0)
+			(at 328.93 136.4746 0)
 			(effects
 				(font
@@
 	)
 	(sheet
-		(at 365.76 181.61)
-		(size 12.7 33.02)
+		(at 328.93 36.83)
+		(size 43.18 44.45)
 		(exclude_from_sim no)
 		(in_bom yes)
@@
 		)
 		(property "Sheetname" "GigbitEthernet"
-			(at 365.76 180.8984 0)
+			(at 328.93 36.1184 0)
 			(effects
 				(font
@@
 		)
 		(property "Sheetfile" "GbEthernet.kicad_sch"
-			(at 365.76 215.2146 0)
+			(at 328.93 81.8646 0)
 			(effects
 				(font
@@
 	)
 	(sheet
-		(at 370.84 284.48)
-		(size 25.4 52.07)
+		(at 194.31 214.63)
+		(size 45.72 69.85)
 		(exclude_from_sim no)
 		(in_bom yes)
@@
 		)
 		(property "Sheetname" "USB 2&3"
-			(at 370.84 283.7684 0)
+			(at 194.31 213.9184 0)
 			(effects
 				(font
@@
 		)
 		(property "Sheetfile" "USB2_3.kicad_sch"
-			(at 370.84 337.1346 0)
+			(at 194.31 285.0646 0)
 			(effects
 				(font
@@
 	)
 	(sheet
-		(at 166.37 177.8)
-		(size 12.7 25.4)
+		(at 194.31 105.41)
+		(size 45.72 100.33)
 		(exclude_from_sim no)
 		(in_bom yes)
@@
 		)
 		(property "Sheetname" "PCIe"
-			(at 166.37 177.0884 0)
+			(at 194.31 104.6984 0)
 			(effects
 				(font
@@
 		)
 		(property "Sheetfile" "PCIe.kicad_sch"
-			(at 166.37 203.7846 0)
+			(at 194.31 206.3246 0)
 			(effects
 				(font
@@
 	)
 	(sheet
-		(at 223.52 212.09)
-		(size 12.7 17.78)
+		(at 194.31 36.83)
+		(size 45.72 22.86)
 		(exclude_from_sim no)
 		(in_bom yes)
@@
 		)
 		(property "Sheetname" "PowerSupply"
-			(at 223.52 211.3784 0)
+			(at 194.31 36.1184 0)
 			(effects
 				(font
@@
 		)
 		(property "Sheetfile" "PowerSupply.kicad_sch"
-			(at 223.52 230.4546 0)
+			(at 194.31 60.2746 0)
 			(effects
 				(font
@@
 	)
 	(sheet
-		(at 250.19 200.66)
-		(size 52.07 83.82)
+		(at 250.19 36.83)
+		(size 69.85 247.65)
 		(exclude_from_sim no)
 		(in_bom yes)
@@
 		)
 		(property "Sheetname" "LaPanda Module"
-			(at 250.19 199.9484 0)
+			(at 250.19 36.1184 0)
 			(effects
 				(font
@@
 	)
 	(sheet
-		(at 430.53 223.52)
-		(size 22.86 59.69)
+		(at 328.93 200.66)
+		(size 43.18 82.55)
 		(exclude_from_sim no)
 		(in_bom yes)
@@
 		)
 		(property "Sheetname" "M2 M Key"
-			(at 430.53 222.8084 0)
+			(at 328.93 199.9484 0)
 			(effects
 				(font
@@
 		)
 		(property "Sheetfile" "M2MKey.kicad_sch"
-			(at 430.53 283.7946 0)
-			(effects
-				(font
+			(at 328.93 283.7946 0)
+			(effects
+				(font

Commit message: Hierachi needs some work
Other:
- sheet Fan ports: added FAN_1_PWM, FAN_1_TAC, FAN_2_PWM, FAN_2_TAC, TEMP; removed none
- sheet GPIO ports: added GPP_D0, GPP_D1, GPP_D2, GPP_D3, I2C2_SCL, I2C2_SDA, I2C3_SCL, I2C3_SDA, I2C4_SCL, I2C4_SDA, I2C5_SCL, I2C5_SDA, SOC_UART0_RX, SOC_UART0_TX, SOC_UART1_RX, SOC_UART1_TX, SOC_UART2_RX, SOC_UART2_TX; removed none
- sheet LaPanda Module ports: added DDI_B_DDC_SCL, DDI_B_DDC_SDA, DDI_B_HPD, DDI_B_TX0+, DDI_B_TX0-, DDI_B_TX1+, DDI_B_TX1-, DDI_B_TX2+, DDI_B_TX2-, DDI_B_TX3+, DDI_B_TX3-, FAN1_PWM, FAN1_TAC, FAN2_PWM, FAN2_TAC, GPP_D0, GPP_D1, GPP_D2, GPP_D3, HSIO_0_RX+, HSIO_0_RX-, HSIO_0_TX+, HSIO_0_TX-, HSIO_10_RX+, HSIO_10_RX-, HSIO_10_TX+, HSIO_10_TX-, HSIO_11_RX+, HSIO_11_RX-, HSIO_11_TX+, HSIO_11_TX-, HSIO_1_RX+, HSIO_1_RX-, HSIO_1_TX+, HSIO_1_TX-, HSIO_2_RX+, HSIO_2_RX-, HSIO_2_TX+, HSIO_2_TX-, HSIO_3_RX+, HSIO_3_RX-, HSIO_3_TX+, HSIO_3_TX-, HSIO_6_RX+, HSIO_6_RX-, HSIO_6_TX+, HSIO_6_TX-, HSIO_8_RX+, HSIO_8_RX-, HSIO_8_TX+, HSIO_8_TX-, HSIO_9_RX+, HSIO_9_RX-, HSIO_9_TX+, HSIO_9_TX-, I2C2_SCL, I2C2_SDA, I2C3_SCL, I2C3_SDA, I2C4_SCL, I2C4_SDA, I2C5_SCL, I2C5_SDA, REFCLK0+, REFCLK0-, REFCLK2+, REFCLK2-, REFCLK3+, REFCLK3-, REFCLK4+, REFCLK4-, SLS_S3, SUSCLK_WIFI, TSENSE, UART0_RXD, UART0_TXD, UART1_RXD, UART1_TXD, UART2_RXD, UART2_TXD, USB2_P1+, USB2_P1-, USB2_P2+, USB2_P2-, USB2_P3+, USB2_P3-, USB2_P4+, USB2_P4-, USB2_P5+, USB2_P5-, USB2_P7+, USB2_P7-, USB2_P8+, USB2_P8-, ~{PLTRST}, ~{PWR_LED}/~{PSON}, ~{PWR_SW}, ~{RST_SW}, ~{WAKE}; removed none
- sheet PCIe ports: added PCIE_RX_0+, PCIE_RX_0-, PCIE_RX_1+, PCIE_RX_1-, PCIE_RX_2+, PCIE_RX_2-, PCIE_RX_3+, PCIE_RX_3-, PCIE_TX_0+, PCIE_TX_0-, PCIE_TX_1+, PCIE_TX_1-, PCIE_TX_2+, PCIE_TX_2-, PCIE_TX_3+, PCIE_TX_3-, PE_RST, REFCLK+, REFCLK-, ~{WAKE}; removed none
- sheet PowerSupply ports: added SLS_S3, ~{PWR_LED}/~{PSON}, ~{PWR_SW}, ~{RST_SW}; removed none

Commit message: fixing Hierachi
Other:
- sheet GigbitEthernet ports: added GbE_PCIe_CLK+, GbE_PCIe_CLK-, GbE_PCIe_RX+, GbE_PCIe_RX-, GbE_PCIe_TX+, GbE_PCIe_TX-, ~{PLT_RST}; removed none
- sheet HDMI ports: added DDI_B_DDC_SCL, DDI_B_DDC_SDA, DDI_B_HPD, DDI_B_TX0+, DDI_B_TX0-, DDI_B_TX1+, DDI_B_TX1-, DDI_B_TX2+, DDI_B_TX2-, DDI_B_TX3+, DDI_B_TX3-, ~{PWR_LED}/~{PSON}; removed none
- sheet LaPanda Module ports: added SCO_UART0_RX, SCO_UART0_TX, SCO_UART1_RX, SCO_UART1_TX, SCO_UART2_RX, SCO_UART2_TX; removed UART0_RXD, UART0_TXD, UART1_RXD, UART1_TXD, UART2_RXD, UART2_TXD
- sheet M2 M Key ports: added PCIE_RX_0+, PCIE_RX_0-, PCIE_RX_1+, PCIE_RX_1-, PCIE_TX_0+, PCIE_TX_0-, PCIE_TX_1+, PCIE_TX_1-, REFCLKE+, REFCLKE-, REFCLKM+, REFCLKM-, SUSCLK, USB_2_P7+, USB_2_P7-, ~{PLT_RST}, ~{WAKE}; removed none
- sheet USB 2&3 ports: added CON_USB1_D_N, CON_USB1_D_P, CON_USB2_D_N, CON_USB2_D_P, USB2_P1+, USB2_P1-, USB2_P2+, USB2_P2-, USB2_P3+, USB2_P3-, USB2_P5+, USB2_P5-, USB3_SSRT_N, USB3_SSRT_P, USB3_SSXT_N, USB3_SSXT_P, USB4_SSRT_N, USB4_SSRT_P, USB4_SSXT_N, USB4_SSXT_P; removed none

Commit message: Still having issues with Hierachi
Other:
- sheet LaPanda Module ports: added none; removed USB2_P4+, USB2_P4-, USB2_P8+, USB2_P8-
- sheet USB 2&3 ports: added none; removed CON_USB1_D_N, CON_USB1_D_P, CON_USB2_D_N, CON_USB2_D_P
Changed lines of the file:
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@@
 		(rev "1")
 	)
-	(rectangle
-		(start 321.31 80.01)
-		(end 326.39 87.63)
-		(stroke
-			(width 0)
-			(type solid)
-			(color 255 69 97 1)
-		)
-		(fill
-			(type none)
-		)
-	)
 	(wire
 		(pts
@@
 	(wire
 		(pts
-			(xy 320.04 80.01) (xy 327.66 80.01)
-		)
-		(stroke
-			(width 0)
-			(type default)
-		)
-	)
-	(wire
-		(pts
 			(xy 320.04 256.54) (xy 328.93 256.54)
 		)
@@
 	(wire
 		(pts
+			(xy 320.04 229.87) (xy 328.93 229.87)
+		)
+		(stroke
+			(width 0)
+			(type default)
+		)
+	)
+	(wire
+		(pts
 			(xy 320.04 171.45) (xy 344.17 171.45)
 		)
@@
 	(wire
 		(pts
-			(xy 320.04 87.63) (xy 327.66 87.63)
-		)
-		(stroke
-			(width 0)
-			(type default)
-		)
-	)
-	(wire
-		(pts
 			(xy 320.04 44.45) (xy 327.66 44.45)
 		)
@@
 	(wire
 		(pts
-			(xy 320.04 82.55) (xy 327.66 82.55)
-		)
-		(stroke
-			(width 0)
-			(type default)
-		)
-	)
-	(wire
-		(pts
 			(xy 240.03 165.1) (xy 250.19 165.1)
 		)
@@
 	(wire
 		(pts
-			(xy 320.04 229.87) (xy 328.93 229.87)
-		)
-		(stroke
-			(width 0)
-			(type default)
-		)
-	)
-	(wire
-		(pts
 			(xy 240.03 153.67) (xy 250.19 153.67)
 		)
@@
 	(wire
 		(pts
-			(xy 320.04 237.49) (xy 328.93 237.49)
-		)
-		(stroke
-			(width 0)
-			(type default)
-		)
-	)
-	(wire
-		(pts
 			(xy 240.03 231.14) (xy 250.19 231.14)
 		)
@@
 	(wire
 		(pts
-			(xy 320.04 85.09) (xy 327.66 85.09)
+			(xy 240.03 138.43) (xy 250.19 138.43)
 		)
 		(stroke
@@
 	(wire
 		(pts
-			(xy 240.03 138.43) (xy 250.19 138.43)
+			(xy 320.04 190.5) (xy 344.17 190.5)
 		)
 		(stroke
@@
 	(wire
 		(pts
-			(xy 320.04 190.5) (xy 344.17 190.5)
+			(xy 240.03 215.9) (xy 250.19 215.9)
 		)
 		(stroke
@@
 	(wire
 		(pts
-			(xy 240.03 215.9) (xy 250.19 215.9)
+			(xy 326.39 142.24) (xy 344.17 142.24)
 		)
 		(stroke
@@
 	(wire
 		(pts
-			(xy 326.39 142.24) (xy 344.17 142.24)
+			(xy 320.04 233.68) (xy 328.93 233.68)
 		)
 		(stroke
@@
 	(wire
 		(pts
-			(xy 320.04 233.68) (xy 328.93 233.68)
+			(xy 240.03 134.62) (xy 250.19 134.62)
 		)
 		(stroke
@@
 	(wire
 		(pts
-			(xy 240.03 134.62) (xy 250.19 134.62)
+			(xy 320.04 245.11) (xy 328.93 245.11)
 		)
 		(stroke
@@
 	(wire
 		(pts
-			(xy 320.04 245.11) (xy 328.93 245.11)
+			(xy 320.04 237.49) (xy 328.93 237.49)
 		)
 		(stroke
@@
 			)
 		)
-		(pin "CON_USB1_D_N" bidirectional
-			(at 327.66 82.55 180)
-			(effects
-				(font
-					(size 1.27 1.27)
-				)
-				(justify left)
-			)
-		)
-		(pin "CON_USB1_D_P" bidirectional
-			(at 327.66 80.01 180)
-			(effects
-				(font
-					(size 1.27 1.27)
-				)
-				(justify left)
-			)
-		)
-		(pin "CON_USB2_D_N" bidirectional
-			(at 327.66 87.63 180)
-			(effects
-				(font
-					(size 1.27 1.27)
-				)
-				(justify left)
-			)
-		)
-		(pin "CON_USB2_D_P" bidirectional
-			(at 327.66 85.09 180)
-			(effects
-				(font
-					(size 1.27 1.27)
-				)
-				(justify left)
-			)
-		)
 		(pin "USB2_P1+" bidirectional
 			(at 327.66 49.53 180)
@@
 		(in_bom yes)
 		(on_board yes)
-		(dnp no)
+		(dnp yes)
 		(fields_autoplaced yes)
 		(stroke
@@
 			)
 		)
-		(pin "HSIO_2_RX+" input
-			(at 320.04 229.87 0)
-			(effects
-				(font
-					(size 1.27 1.27)
-				)
-				(justify right)
-			)
-		)
-		(pin "HSIO_2_RX-" input
-			(at 320.04 233.68 0)
-			(effects
-				(font
-					(size 1.27 1.27)
-				)
-				(justify right)
-			)
-		)
-		(pin "HSIO_2_TX+" output
-			(at 320.04 237.49 0)
-			(effects
-				(font
-					(size 1.27 1.27)
-				)
-				(justify right)
-			)
-		)
-		(pin "HSIO_2_TX-" output
-			(at 320.04 241.3 0)
-			(effects
-				(font
-					(size 1.27 1.27)
-				)
-				(justify right)
-			)
-		)
 		(pin "HSIO_3_RX+" input
 			(at 320.04 214.63 0)
@@
 			)
 		)
-		(pin "USB2_P4+" bidirectional
-			(at 320.04 80.01 0)
-			(effects
-				(font
-					(size 1.27 1.27)
-				)
-				(justify right)
-			)
-		)
-		(pin "USB2_P4-" bidirectional
-			(at 320.04 82.55 0)
-			(effects
-				(font
-					(size 1.27 1.27)
-				)
-				(justify right)
-			)
-		)
 		(pin "USB2_P5+" bidirectional
 			(at 320.04 64.77 0)
@@
 			)
 		)
-		(pin "USB2_P8+" bidirectional
-			(at 320.04 85.09 0)
-			(effects
-				(font
-					(size 1.27 1.27)
-				)
-				(justify right)
-			)
-		)
-		(pin "USB2_P8-" input
-			(at 320.04 87.63 0)
-			(effects
-				(font
-					(size 1.27 1.27)
-				)
-				(justify right)
-			)
-		)
 		(pin "~{PLTRST}" output
 			(at 250.19 181.61 180)
@@
 			)
 		)
+		(pin "HSIO_2_RX+" input
+			(at 320.04 229.87 0)
+			(effects
+				(font
+					(size 1.27 1.27)
+				)
+				(justify right)
+			)
+		)
+		(pin "HSIO_2_RX-" input
+			(at 320.04 233.68 0)
+			(effects
+				(font
+					(size 1.27 1.27)
+				)
+				(justify right)
+			)
+		)
+		(pin "HSIO_2_TX+" output
+			(at 320.04 237.49 0)
+			(effects
+				(font
+					(size 1.27 1.27)
+				)
+				(justify right)
+			)
+		)
+		(pin "HSIO_2_TX-" output
+			(at 320.04 241.3 0)
+			(effects
+				(font
+					(size 1.27 1.27)
+				)
+				(justify right)
+			)
+		)
 		(instances
 			(project "LattepndaCourse"
@@
 			)
 		)
-		(pin "PCIE_RX_1+" output
-			(at 328.93 229.87 180)
+		(pin "PCIE_TX_0+" input
+			(at 328.93 222.25 180)
 			(effects
 				(font
@@
 			)
 		)
-		(pin "PCIE_RX_1-" output
-			(at 328.93 233.68 180)
+		(pin "PCIE_TX_0-" input
+			(at 328.93 226.06 180)
 			(effects
 				(font
@@
 			)
 		)
-		(pin "PCIE_TX_0+" input
-			(at 328.93 222.25 180)
+		(pin "REFCLKE+" bidirectional
+			(at 328.93 245.11 180)
 			(effects
 				(font
@@
 			)
 		)
-		(pin "PCIE_TX_0-" input
-			(at 328.93 226.06 180)
+		(pin "REFCLKE-" bidirectional
+			(at 328.93 248.92 180)
 			(effects
 				(font
@@
 			)
 		)
-		(pin "PCIE_TX_1+" input
-			(at 328.93 237.49 180)
+		(pin "REFCLKM+" output
+			(at 328.93 252.73 180)
 			(effects
 				(font
@@
 			)
 		)
-		(pin "PCIE_TX_1-" input
-			(at 328.93 241.3 180)
+		(pin "REFCLKM-" output
+			(at 328.93 256.54 180)
 			(effects
 				(font
@@
 			)
 		)
-		(pin "REFCLKE+" bidirectional
-			(at 328.93 245.11 180)
+		(pin "SUSCLK" output
+			(at 328.93 262.89 180)
 			(effects
 				(font
@@
 			)
 		)
-		(pin "REFCLKE-" bidirectional
-			(at 328.93 248.92 180)
+		(pin "USB_2_P7+" bidirectional
+			(at 328.93 266.7 180)
 			(effects
 				(font
@@
 			)
 		)
-		(pin "REFCLKM+" output
-			(at 328.93 252.73 180)
+		(pin "USB_2_P7-" bidirectional
+			(at 328.93 270.51 180)
 			(effects
 				(font
@@
 			)
 		)
-		(pin "REFCLKM-" output
-			(at 328.93 256.54 180)
+		(pin "~{PLT_RST}" input
+			(at 328.93 274.32 180)
 			(effects
 				(font
@@
 			)
 		)
-		(pin "SUSCLK" output
-			(at 328.93 262.89 180)
+		(pin "~{WAKE}" input
+			(at 328.93 278.13 180)
 			(effects
 				(font
@@
 			)
 		)
-		(pin "USB_2_P7+" bidirectional
-			(at 328.93 266.7 180)
+		(pin "PCIE_RX_1+" output
+			(at 328.93 229.87 180)
 			(effects
 				(font
@@
 			)
 		)
-		(pin "USB_2_P7-" bidirectional
-			(at 328.93 270.51 180)
+		(pin "PCIE_RX_1-" output
+			(at 328.93 233.68 180)
 			(effects
 				(font
@@
 			)
 		)
-		(pin "~{PLT_RST}" input
-			(at 328.93 274.32 180)
+		(pin "PCIE_TX_1+" input
+			(at 328.93 237.49 180)
 			(effects
 				(font
@@
 			)
 		)
-		(pin "~{WAKE}" input
-			(at 328.93 278.13 180)
+		(pin "PCIE_TX_1-" input
+			(at 328.93 241.3 180)
 			(effects
 				(font
