File: project1/LattepndaCourse/Fan.kicad_sch (KiCad schematic)
At the start: 0 parts

Commit message: Hierachi
Other:
- title: (none) -> practice design
Changed lines of the file:
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@@
 	(generator "eeschema")
 	(generator_version "9.0")
-	(paper "A4")
+	(paper "A2")
+	(title_block
+		(title "practice design")
+		(date "2026-09-30")
+		(rev "1")
+	)
 )

Commit message: working on GPIO
Parts:
- added C24, C25: 100nF/50V, A_HDJ_Library:C_0402_1005Metric, symbol Device:C_Small
- added D17, D18: 1N5819WS, A_HDJ_Library:D_SOD-323, symbol Diode:1N5819WS
- added JP2: NTC_Test, Jumper:SolderJumper-2_P1.3mm_Open_RoundedPad1.0x1.5mm, symbol Jumper:SolderJumper_2_Open
- added M1, M2: Fan_4pin, A_HDJ_Library:JST_PH_B4B-PH-K_1x04_P2.00mm_Vertical, symbol Motor:Fan_4pin
- added R32, R37, R38, R40: 4.7K/1%, A_HDJ_Library:R_0402_1005Metric, symbol Device:R
- added R33, R35, R39, R41: 21.5K/1%, A_HDJ_Library:R_0402_1005Metric, symbol Device:R
- added R34, R36: 100R/1%, A_HDJ_Library:R_0402_1005Metric, symbol Device:R
- added R42, R43: 0R/1%, A_HDJ_Library:R_0402_1005Metric, symbol Device:R
- added R44: 10K/1%, A_HDJ_Library:R_0402_1005Metric, symbol Device:R
- added TH1: NTC-10K, A_HDJ_Library:R_0603_1608Metric, symbol Device:Thermistor_NTC
- added TP10, TP11, TP12, TP9: TestPoint, symbol Connector:TestPoint
Connections:
- new net: C25.1, D18.1 (K), M2.2 (+), R37.2, R42.1, R43.1
- new net: D18.2 (A), M2.3 (Tacho), R35.1, R37.1
- new net: M2.4 (PWM), R36.1
- new net: D17.2 (A), M1.3 (Tacho), R32.1, R33.1
- new net: JP2.2 (B), R44.2, TH1.1
- new net: M1.4 (PWM), R34.1
- new net +12V: R43.2
- new net +3V3: R38.2, R44.1
- new net +5V: C24.1, D17.1 (K), M1.2 (+), R32.2, R42.2
- new net FAN_1_PWM: R34.2, R38.1, TP9.1
- new net FAN_1_TAC: R33.2, R39.1, TP10.1
- new net FAN_2_PWM: R36.2, R40.1, TP11.1
- new net FAN_2_TAC: R35.2, R41.1, TP12.1
- new net GND: C24.2, C25.2, M1.1 (-), M2.1 (-), R39.2, R41.2, TH1.2
- new net TEMP: JP2.1 (A)
Other:
- note added: "CPU FAN"
- note added: "LattePanda has Pull-Up resistors"
- note added: "Reversed for 12V fan FAN_TAC input only allows 3.3V level"
- note added: "SYS FAN"

Commit message: USB is done
Changed lines of the file:
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@@
 	(wire
 		(pts
-			(xy 57.15 111.76) (xy 64.77 111.76)
+			(xy 58.42 111.76) (xy 64.77 111.76)
 		)
 		(stroke
@@
 	(global_label "TEMP"
 		(shape output)
-		(at 57.15 111.76 180)
+		(at 58.42 111.76 180)
 		(fields_autoplaced yes)
 		(effects
@@
 		)
 		(property "Intersheetrefs" "${INTERSHEET_REFS}"
-			(at 49.3268 111.76 0)
+			(at 50.5968 111.76 0)
 			(hide yes)
 			(show_name no)

Commit message: Hierachi needs some work
Connections:
- net +3V3: now also R40.2
Changed lines of the file:
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@@
 		)
 	)
-	(global_label "FAN_2_PWM"
+	(wire
+		(pts
+			(xy 151.13 124.46) (xy 151.13 127)
+		)
+		(stroke
+			(width 0)
+			(type default)
+		)
+	)
+	(hierarchical_label "FAN_1_PWM"
 		(shape input)
-		(at 143.51 142.24 180)
-		(fields_autoplaced yes)
+		(at 143.51 69.85 180)
 		(effects
 			(font
@@
 			(justify right)
 		)
-		(property "Intersheetrefs" "${INTERSHEET_REFS}"
-			(at 129.6996 142.24 0)
-			(hide yes)
-			(show_name no)
-			(do_not_autoplace no)
-			(effects
-				(font
-					(size 1.27 1.27)
-				)
-				(justify right)
-			)
-		)
-	)
-	(global_label "TEMP"
+	)
+	(hierarchical_label "TEMP"
 		(shape output)
 		(at 58.42 111.76 180)
-		(fields_autoplaced yes)
 		(effects
 			(font
@@
 			(justify right)
 		)
-		(property "Intersheetrefs" "${INTERSHEET_REFS}"
-			(at 50.5968 111.76 0)
-			(hide yes)
-			(show_name no)
-			(do_not_autoplace no)
-			(effects
-				(font
-					(size 1.27 1.27)
-				)
-				(justify right)
-			)
-		)
-	)
-	(global_label "FAN_1_TAC"
-		(shape output)
-		(at 142.24 64.77 180)
-		(fields_autoplaced yes)
+	)
+	(hierarchical_label "FAN_2_TAC"
+		(shape input)
+		(at 142.24 137.16 180)
 		(effects
 			(font
@@
 			(justify right)
 		)
-		(property "Intersheetrefs" "${INTERSHEET_REFS}"
-			(at 129.2762 64.77 0)
-			(hide yes)
-			(show_name no)
-			(do_not_autoplace no)
-			(effects
-				(font
-					(size 1.27 1.27)
-				)
-				(justify right)
-			)
-		)
-	)
-	(global_label "FAN_2_TAC"
-		(shape output)
-		(at 142.24 137.16 180)
-		(fields_autoplaced yes)
+	)
+	(hierarchical_label "FAN_2_PWM"
+		(shape input)
+		(at 143.51 142.24 180)
 		(effects
 			(font
@@
 			(justify right)
 		)
-		(property "Intersheetrefs" "${INTERSHEET_REFS}"
-			(at 129.2762 137.16 0)
-			(hide yes)
-			(show_name no)
-			(do_not_autoplace no)
-			(effects
-				(font
-					(size 1.27 1.27)
-				)
-				(justify right)
-			)
-		)
-	)
-	(global_label "FAN_1_PWM"
+	)
+	(hierarchical_label "FAN_1_TAC"
 		(shape input)
-		(at 143.51 69.85 180)
-		(fields_autoplaced yes)
+		(at 142.24 64.77 180)
 		(effects
 			(font
@@
 			)
 			(justify right)
-		)
-		(property "Intersheetrefs" "${INTERSHEET_REFS}"
-			(at 129.6996 69.85 0)
-			(hide yes)
-			(show_name no)
-			(do_not_autoplace no)
-			(effects
-				(font
-					(size 1.27 1.27)
-				)
-				(justify right)
-			)
 		)
 	)
@@
 					(unit 1)
 				)
+			)
+		)
+	)
+	(symbol
+		(lib_id "power:+5V")
+		(at 151.13 124.46 0)
+		(unit 1)
+		(body_style 1)
+		(exclude_from_sim no)
+		(in_bom yes)
+		(on_board yes)
+		(in_pos_files yes)
+		(dnp no)
+		(fields_autoplaced yes)
+		(property "Reference" "#PWR0121"
+			(at 151.13 128.27 0)
+			(hide yes)
+			(show_name no)
+			(do_not_autoplace no)
+			(effects
+				(font
+					(size 1.27 1.27)
+				)
+			)
+		)
+		(property "Value" "+3V3"
+			(at 151.13 119.38 0)
+			(show_name no)
+			(do_not_autoplace no)
+			(effects
+				(font
+					(size 1.27 1.27)
+				)
+			)
+		)
+		(property "Footprint" ""
+			(at 151.13 124.46 0)
+			(hide yes)
+			(show_name no)
+			(do_not_autoplace no)
+			(effects
+				(font
+					(size 1.27 1.27)
+				)
+			)
+		)
+		(property "Datasheet" ""
+			(at 151.13 124.46 0)
+			(hide yes)
+			(show_name no)
+			(do_not_autoplace no)
+			(effects
+				(font
+					(size 1.27 1.27)
+				)
+			)
+		)
+		(property "Description" "Power symbol creates a global label with name \"+5V\""
+			(at 151.13 124.46 0)
+			(hide yes)
+			(show_name no)
+			(do_not_autoplace no)
+			(effects
+				(font
+					(size 1.27 1.27)
+				)
+			)
+		)
+		(pin "1"
+		)
+		(instances
+			(project "LattepndaCourse"
+				(path "/4e04f3a7-ba43-4db9-8bbc-1a27efcf5abf/259c3d94-424d-4775-b548-b0cce5d71fc7"
+					(reference "#PWR0121")
+					(unit 1)
+				)

Commit message: Started routing
Parts:
- TP10, TP11, TP12, TP9: footprint (none) -> A_HDJ_Library:TestPoint_Pad_D1.5mm
