File: project1/LattepndaCourse/GbEthernet.kicad_sch (KiCad schematic)
At the start: 0 parts

Commit message: Hierachi
Other:
- title: (none) -> practice design
Changed lines of the file:
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@@
 	(generator "eeschema")
 	(generator_version "9.0")
-	(paper "A4")
+	(paper "A2")
+	(title_block
+		(title "practice design")
+		(date "2026-09-30")
+		(rev "1")
+	)
 )

Commit message: Gigbit Ethernet is done
Parts:
- added C33, C44, C45, C46, C47, C48, C50, C51, C52, C53, C54, C55, C56: 100nF/50V, A_HDJ_Library:C_0402_1005Metric, symbol Device:C_Small
- added C42, C43: 12pF/50V, A_HDJ_Library:C_0402_1005Metric, symbol Device:C_Small
- added C49: 10uF/50V, A_HDJ_Library:C_0402_1005Metric, symbol Device:C_Small
- added J15: RJ45_RB1-125B8G1A, A_HDJ_Library:RJ45_UDE_RB1-125B8G1A, symbol Connector:RJ45_RB1-125B8G1A
- added R45, R46: 470R/1%, A_HDJ_Library:R_0402_1005Metric, symbol Device:R
- added R47: 1M/1%, A_HDJ_Library:R_0402_1005Metric, symbol Device:R
- added R48: 2.49K/1%, A_HDJ_Library:R_0603_1608Metric, symbol Device:R
- added R49, R50: 10K/1%, A_HDJ_Library:R_0402_1005Metric, symbol Device:R
- added U10: RTL8111H-CG-RH, A_HDJ_Library:QFN-32-1EP_4x4mm_P0.4mm_EP2.65x2.65mm, symbol A_HDJ_Library:RTL8111H-CG-RH
- added U11, U12: ULC0524P, A_HDJ_Library:Diodes_UDFN-10_1.0x2.5mm_P0.5mm, symbol Power_Protection:D3V3XA4B10LP
- added Y1: 25MHz, symbol Device:Crystal_GND24
Connections:
- new net: R49.1, U10.20 (ISOLATEB)
- new net: R48.2, U10.31 (RSET)
- new net: J15.L1, R46.2
- new net: C33.2, J15.R1 (CT)
- new net: C43.1, R47.2, U10.28 (CKXTAL1), Y1.1
- new net: C42.1, R47.1, U10.29 (CKXTAL2), Y1.3
- new net: J15.L3, R45.2
- new net: J15.L2, U10.25 (LED2)
- new net: J15.L4, U10.26 (LED1)
- new net: R50.1, U10.21 (LANWAKEB)
- new net +1V0: C44.1, C45.1, C46.1, C47.1, C48.1, C49.1, U10.22 (DVDD10), U10.24 (REGOUT), U10.3 (AVDD10), U10.30 (AVDD10), U10.8 (AVDD10)
- new net +3.3V: C50.1, C51.1, C52.1, R45.1, R46.1, R49.2, R50.2, U10.11 (AVDD33)
- new net GND: C33.1, C42.2, C43.2, C44.2, C45.2, C46.2, C47.2, C48.2, C49.2, C50.2, C51.2, C52.2, J15.R10 (GND), J15.SH, R48.1, U10.12 (CLKREQB), U10.33 (GND), U11.3 (VSS), U11.8 (VSS), U12.3 (VSS), U12.8 (VSS), Y1.2 (G), Y1.4 (G)
- new net GbE_PCIe_CLK+: U10.15 (REFCLK_P)
- new net GbE_PCIe_CLK-: U10.16 (REFCLK_N)
- new net GbE_PCIe_RX+: C56.1
- new net GbE_PCIe_RX-: C55.1
- new net GbE_PCIe_TX+: C54.1
- new net GbE_PCIe_TX-: C53.1
- new net HSI+: C54.2, U10.13 (HSIP)
- new net HSI-: C53.2, U10.14 (HSIN)
- new net HSO+: C56.2, U10.17 (HSOP)
- new net HSO-: C55.2, U10.18 (HSON)
- new net MDI0+: J15.R2 (TD1+), U10.1 (MDIP0), U12.4, U12.7 (NC)
- new net MDI0-: J15.R3 (TD1-), U10.2 (MDIN0), U12.5, U12.6 (NC)
- new net MDI1+: J15.R4 (TD2+), U10.4 (MDIP1), U12.1, U12.10 (NC)
- new net MDI1-: J15.R5 (TD2-), U10.5 (MDIN1), U12.2, U12.9 (NC)
- new net MDI2+: J15.R6 (TD3+), U10.6 (MDIP2), U11.5, U11.6 (NC)
- new net MDI2-: J15.R7 (TD3-), U10.7 (MDIN2), U11.4, U11.7 (NC)
- new net MDI3+: J15.R8 (TD4+), U10.9 (MDIP3), U11.2, U11.9 (NC)
- new net MDI3-: J15.R9 (TD4-), U10.10 (MDIN3), U11.1, U11.10 (NC)
- new net ~{PLT_RST}: U10.19 (PERSTB)

Commit message: USB is done
Connections:
- no-connect marks 0 -> 3
Changed lines of the file:
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@@
 		(color 0 0 0 0)
+	)
+	(no_connect
+		(at 130.81 118.11)
+	)
+	(no_connect
+		(at 99.06 88.9)
+	)
+	(no_connect
+		(at 99.06 91.44)
 	)
 	(wire

Commit message: fixing Hierachi
Changed lines of the file:
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@@
 		)
 	)
-	(global_label "GbE_PCIe_CLK+"
-		(shape input)
-		(at 53.34 130.81 180)
-		(fields_autoplaced yes)
+	(hierarchical_label "GbE_PCIe_RX+"
+		(shape output)
+		(at 53.34 125.73 180)
 		(effects
 			(font
@@
 			(justify right)
 		)
-		(property "Intersheetrefs" "${INTERSHEET_REFS}"
-			(at 35.4777 130.81 0)
-			(hide yes)
-			(show_name no)
-			(do_not_autoplace no)
-			(effects
-				(font
-					(size 1.27 1.27)
-				)
-				(justify right)
-			)
-		)
 	)
-	(global_label "~{PLT_RST}"
+	(hierarchical_label "GbE_PCIe_TX+"
 		(shape input)
-		(at 53.34 133.35 180)
-		(fields_autoplaced yes)
+		(at 53.34 120.65 180)
 		(effects
 			(font
@@
 			(justify right)
 		)
-		(property "Intersheetrefs" "${INTERSHEET_REFS}"
-			(at 42.6744 133.35 0)
-			(hide yes)
-			(show_name no)
-			(do_not_autoplace no)
-			(effects
-				(font
-					(size 1.27 1.27)
-				)
-				(justify right)
-			)
-		)
 	)
-	(global_label "GbE_PCIe_RX-"
-		(shape output)
-		(at 53.34 123.19 180)
-		(fields_autoplaced yes)
+	(hierarchical_label "GbE_PCIe_CLK-"
+		(shape input)
+		(at 53.34 128.27 180)
 		(effects
 			(font
@@
 			(justify right)
 		)
-		(property "Intersheetrefs" "${INTERSHEET_REFS}"
-			(at 36.5663 123.19 0)
-			(hide yes)
-			(show_name no)
-			(do_not_autoplace no)
-			(effects
-				(font
-					(size 1.27 1.27)
-				)
-				(justify right)
-			)
-		)
 	)
-	(global_label "GbE_PCIe_CLK-"
+	(hierarchical_label "~{PLT_RST}"
 		(shape input)
-		(at 53.34 128.27 180)
-		(fields_autoplaced yes)
+		(at 53.34 133.35 180)
 		(effects
 			(font
@@
 			(justify right)
 		)
-		(property "Intersheetrefs" "${INTERSHEET_REFS}"
-			(at 35.4777 128.27 0)
-			(hide yes)
-			(show_name no)
-			(do_not_autoplace no)
-			(effects
-				(font
-					(size 1.27 1.27)
-				)
-				(justify right)
-			)
-		)
 	)
-	(global_label "GbE_PCIe_TX+"
+	(hierarchical_label "GbE_PCIe_TX-"
 		(shape input)
-		(at 53.34 120.65 180)
-		(fields_autoplaced yes)
+		(at 53.34 118.11 180)
 		(effects
 			(font
@@
 			(justify right)
 		)
-		(property "Intersheetrefs" "${INTERSHEET_REFS}"
-			(at 36.8687 120.65 0)
-			(hide yes)
-			(show_name no)
-			(do_not_autoplace no)
-			(effects
-				(font
-					(size 1.27 1.27)
-				)
-				(justify right)
-			)
-		)
 	)
-	(global_label "GbE_PCIe_TX-"
-		(shape input)
-		(at 53.34 118.11 180)
-		(fields_autoplaced yes)
+	(hierarchical_label "GbE_PCIe_RX-"
+		(shape output)
+		(at 53.34 123.19 180)
 		(effects
 			(font
@@
 			(justify right)
 		)
-		(property "Intersheetrefs" "${INTERSHEET_REFS}"
-			(at 36.8687 118.11 0)
-			(hide yes)
-			(show_name no)
-			(do_not_autoplace no)
-			(effects
-				(font
-					(size 1.27 1.27)
-				)
-				(justify right)
-			)
-		)
 	)
-	(global_label "GbE_PCIe_RX+"
-		(shape output)
-		(at 53.34 125.73 180)
-		(fields_autoplaced yes)
+	(hierarchical_label "GbE_PCIe_CLK+"
+		(shape input)
+		(at 53.34 130.81 180)
 		(effects
 			(font
@@
 			(justify right)
 		)
-		(property "Intersheetrefs" "${INTERSHEET_REFS}"
-			(at 36.5663 125.73 0)
-			(hide yes)
-			(show_name no)
-			(do_not_autoplace no)
-			(effects
-				(font
-					(size 1.27 1.27)
-				)
-				(justify right)
-			)
-		)
 	)

Commit message: Started routing
Parts:
- Y1: footprint (none) -> A_HDJ_Library:Crystal_SMD_3225-4Pin_3.2x2.5mm
