File: project1/LattepndaCourse/HDMI.kicad_sch (KiCad schematic)
At the start: 0 parts

Commit message: Hierachi
Other:
- title: (none) -> practice design
Changed lines of the file:
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@@
 	(generator "eeschema")
 	(generator_version "9.0")
-	(paper "A4")
+	(paper "A2")
+	(title_block
+		(title "practice design")
+		(date "2026-09-30")
+		(rev "1")
+	)
 )

Commit message: cont HDMI
Parts:
- added C63, C64, C65, C66, C67, C68, C69, C70: 100nF/50V, A_HDJ_Library:C_0603_1608Metric, symbol Device:C_Small
- added J19: HDMI_A, A_HDJ_Library:HDMI_A_Molex_208658-1001_Horizontal, symbol Connector:HDMI_A
- added Q6, Q7, Q9: 2SK3018, A_HDJ_Library:SOT-23, symbol Transistor_FET:2N7002
- added Q8: 2N7002, A_HDJ_Library:SOT-23, symbol Transistor_FET:2N7002
- added R51, R52, R53, R54, R55, R56, R57, R58: 470R/1%, A_HDJ_Library:R_0402_1005Metric, symbol Device:R
- added R59: 2.5K/1%, A_HDJ_Library:R_0402_1005Metric, symbol Device:R
- added R60, R61: 2.2K/1%, A_HDJ_Library:R_0402_1005Metric, symbol Device:R
- added U16, U17: ULC0524P, A_HDJ_Library:Diodes_UDFN-10_1.0x2.5mm_P0.5mm, symbol Power_Protection:D3V3XA4B10LP
Connections:
- new net: Q9.3 (D), R51.1, R52.1, R53.1, R54.1, R55.1, R56.1, R57.1, R58.1
- new net: J19.15 (SCL), Q6.2 (S)
- new net: J19.16 (SDA), Q7.2 (S)
- new net: J19.19 (HPD), Q8.2 (S)
- new net: Q9.1 (G), R59.2
- new net +3V3: R60.1, R61.1
- new net DDI_B_DDC_SCL: Q6.3 (D), R61.2
- new net DDI_B_DDC_SDA: Q7.3 (D), R60.2
- new net DDI_B_TX0+: C63.2, C69.2
- new net DDI_B_TX0-: C64.2, C70.2
- new net DDI_B_TX1+: C65.2
- new net DDI_B_TX1-: C66.2
- new net DDI_B_TX2+: C67.2
- new net DDI_B_TX2-: C68.2
- new net GND: J19.11 (CKS), J19.17 (GND), J19.2 (D2S), J19.5 (D1S), J19.8 (D0S), J19.SH, Q9.2 (S), U16.3 (VSS), U16.8 (VSS), U17.3 (VSS), U17.8 (VSS)
- new net TMDS_CK+: C69.1, J19.10 (CK+), R52.2, U17.4, U17.7 (NC)
- new net TMDS_CK-: C70.1, J19.12 (CK-), R51.2, U17.5, U17.6 (NC)
- new net TMDS_D0+: C67.1, J19.7 (D0+), R54.2, U17.1, U17.10 (NC)
- new net TMDS_D0-: C68.1, J19.9 (D0-), R53.2, U17.2, U17.9 (NC)
- new net TMDS_D1+: C65.1, J19.4 (D1+), R56.2, U16.4, U16.7 (NC)
- new net TMDS_D1-: C66.1, J19.6 (D1-), R55.2, U16.5, U16.6 (NC)
- new net TMDS_D2+: C63.1, J19.1 (D2+), R58.2, U16.1, U16.10 (NC)
- new net TMDS_D2-: C64.1, J19.3 (D2-), R57.2, U16.2, U16.9 (NC)
- new net ~{PWR_LED}/~{PSON}: R59.1

Commit message: HDMI is done
Parts:
- added C71: 100nF/50V, A_HDJ_Library:C_0603_1608Metric, symbol Device:C_Small
- added D23: 1N5819WS, A_HDJ_Library:D_SOD-323, symbol Diode:1N5819WS
- added D24, D25, D26: ESD5V0B03, A_HDJ_Library:D_0402_1005Metric, symbol Diode:ESD9B5.0ST5G
- added F5: 6V/50mA, A_HDJ_Library:C_0603_1608Metric, symbol Device:Fuse
- added R62, R63: 2.2K/1%, A_HDJ_Library:R_0402_1005Metric, symbol Device:R
- added R64: 1M/1%, A_HDJ_Library:R_0402_1005Metric, symbol Device:R
- added R66: 1K/1%, A_HDJ_Library:R_0402_1005Metric, symbol Device:R
- added R67: 21.5K/1%, A_HDJ_Library:R_0402_1005Metric, symbol Device:R
Connections:
- net +3V3: now also Q6.1 (G), Q7.1 (G), Q8.1 (G), R64.1
- net GND: now also C71.2, D24.1 (A1), D25.1 (A1), D26.1 (A1), R67.2
- net DDC_SCL: now reaches J19.15 (SCL), Q6.2 (S)
- net DDC_SCL: now also D25.2 (A2), R62.2
- net DDC_SDA: now reaches J19.16 (SDA), Q7.2 (S)
- net DDC_SDA: now also D24.2 (A2), R63.2
- net at J19.18 (+5V): now also F5.2
- net at Q8.2 (S): now also R66.1, R67.1; no longer J19.19 (HPD)
- net DDI_B_HPD: now reaches Q8.3 (D)
- net DDI_B_HPD: now also R64.2
- new net +5V: D23.2 (A)
- new net 5V_HDMI_VCC: C71.1, D23.1 (K), F5.1, R62.1, R63.1
- new net HPD: D26.2 (A2), J19.19 (HPD), R66.2
- no-connect marks 0 -> 2
Other:
- moved on the sheet: Q6, Q7, Q8, R60, R61

Commit message: fixing Hierachi
Connections:
- net DDI_B_TX0+: no longer C69.2
- net DDI_B_TX0-: no longer C70.2
- new net DDI_B_TX3+: C69.2
- new net DDI_B_TX3-: C70.2
Changed lines of the file:
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@@
 		)
 	)
-	(global_label "DDI_B_TX1+"
+	(hierarchical_label "DDI_B_TX2+"
 		(shape input)
-		(at 125.73 57.15 180)
-		(fields_autoplaced yes)
+		(at 125.73 62.23 180)
 		(effects
 			(font
@@
 			(justify right)
 		)
-		(property "Intersheetrefs" "${INTERSHEET_REFS}"
-			(at 111.4358 57.15 0)
-			(hide yes)
-			(show_name no)
-			(do_not_autoplace no)
-			(effects
-				(font
-					(size 1.27 1.27)
-				)
-				(justify right)
-			)
-		)
 	)
-	(global_label "DDI_B_TX1-"
-		(shape input)
-		(at 125.73 59.69 180)
-		(fields_autoplaced yes)
+	(hierarchical_label "DDI_B_DDC_SCL"
+		(shape output)
+		(at 96.52 119.38 180)
 		(effects
 			(font
@@
 			(justify right)
 		)
-		(property "Intersheetrefs" "${INTERSHEET_REFS}"
-			(at 111.4358 59.69 0)
-			(hide yes)
-			(show_name no)
-			(do_not_autoplace no)
-			(effects
-				(font
-					(size 1.27 1.27)
-				)
-				(justify right)
-			)
-		)
 	)
-	(global_label "DDI_B_TX0+"
+	(hierarchical_label "DDI_B_TX3-"
 		(shape input)
-		(at 125.73 67.31 180)
-		(fields_autoplaced yes)
+		(at 125.73 69.85 180)
 		(effects
 			(font
@@
 			(justify right)
 		)
-		(property "Intersheetrefs" "${INTERSHEET_REFS}"
-			(at 111.4358 67.31 0)
-			(hide yes)
-			(show_name no)
-			(do_not_autoplace no)
-			(effects
-				(font
-					(size 1.27 1.27)
-				)
-				(justify right)
-			)
-		)
 	)
-	(global_label "DDI_B_TX2-"
+	(hierarchical_label "DDI_B_TX0+"
 		(shape input)
-		(at 125.73 64.77 180)
-		(fields_autoplaced yes)
+		(at 125.73 52.07 180)
 		(effects
 			(font
@@
 			(justify right)
 		)
-		(property "Intersheetrefs" "${INTERSHEET_REFS}"
-			(at 111.4358 64.77 0)
-			(hide yes)
-			(show_name no)
-			(do_not_autoplace no)
-			(effects
-				(font
-					(size 1.27 1.27)
-				)
-				(justify right)
-			)
-		)
 	)
-	(global_label "DDI_B_DDC_SDA"
+	(hierarchical_label "DDI_B_DDC_SDA"
 		(shape bidirectional)
 		(at 97.79 135.89 180)
-		(fields_autoplaced yes)
 		(effects
 			(font
@@
 			(justify right)
 		)
-		(property "Intersheetrefs" "${INTERSHEET_REFS}"
-			(at 78.9978 135.89 0)
-			(hide yes)
-			(show_name no)
-			(do_not_autoplace no)
-			(effects
-				(font
-					(size 1.27 1.27)
-				)
-				(justify right)
+	)
+	(hierarchical_label "DDI_B_TX1+"
+		(shape input)
+		(at 125.73 57.15 180)
+		(effects
+			(font
+				(size 1.27 1.27)
 			)
+			(justify right)
 		)
 	)
-	(global_label "~{PWR_LED}{slash}~{PSON}"
+	(hierarchical_label "DDI_B_TX3+"
+		(shape input)
+		(at 125.73 67.31 180)
+		(effects
+			(font
+				(size 1.27 1.27)
+			)
+			(justify right)
+		)
+	)
+	(hierarchical_label "DDI_B_TX1-"
+		(shape input)
+		(at 125.73 59.69 180)
+		(effects
+			(font
+				(size 1.27 1.27)
+			)
+			(justify right)
+		)
+	)
+	(hierarchical_label "DDI_B_TX2-"
+		(shape input)
+		(at 125.73 64.77 180)
+		(effects
+			(font
+				(size 1.27 1.27)
+			)
+			(justify right)
+		)
+	)
+	(hierarchical_label "~{PWR_LED}{slash}~{PSON}"
 		(shape input)
 		(at 224.79 101.6 0)
-		(fields_autoplaced yes)
 		(effects
 			(font
@@
 			(justify left)
 		)
-		(property "Intersheetrefs" "${INTERSHEET_REFS}"
-			(at 242.6523 101.6 0)
-			(hide yes)
-			(show_name no)
-			(do_not_autoplace no)
-			(effects
-				(font
-					(size 1.27 1.27)
-				)
-				(justify left)
-			)
-		)
 	)
-	(global_label "DDI_B_TX2+"
+	(hierarchical_label "DDI_B_TX0-"
 		(shape input)
-		(at 125.73 62.23 180)
-		(fields_autoplaced yes)
+		(at 125.73 54.61 180)
 		(effects
 			(font
@@
 			(justify right)
 		)
-		(property "Intersheetrefs" "${INTERSHEET_REFS}"
-			(at 111.4358 62.23 0)
-			(hide yes)
-			(show_name no)
-			(do_not_autoplace no)
-			(effects
-				(font
-					(size 1.27 1.27)
-				)
-				(justify right)
-			)
-		)
 	)
-	(global_label "DDI_B_TX0+"
+	(hierarchical_label "DDI_B_HPD"
 		(shape input)
-		(at 125.73 52.07 180)
-		(fields_autoplaced yes)
+		(at 92.71 156.21 180)
 		(effects
 			(font
@@
 			(justify right)
 		)
-		(property "Intersheetrefs" "${INTERSHEET_REFS}"
-			(at 111.4358 52.07 0)
-			(hide yes)
-			(show_name no)
-			(do_not_autoplace no)
-			(effects
-				(font
-					(size 1.27 1.27)
-				)
-				(justify right)
-			)
-		)
 	)
-	(global_label "DDI_B_TX0-"
-		(shape input)
-		(at 125.73 54.61 180)
-		(fields_autoplaced yes)
-		(effects
-			(font
-				(size 1.27 1.27)
-			)
-			(justify right)
-		)
-		(property "Intersheetrefs" "${INTERSHEET_REFS}"
-			(at 111.4358 54.61 0)
-			(hide yes)
-			(show_name no)
-			(do_not_autoplace no)
-			(effects
-				(font
-					(size 1.27 1.27)
-				)
-				(justify right)
-			)
-		)
-	)
-	(global_label "DDI_B_DDC_SCL"
-		(shape output)
-		(at 96.52 119.38 180)
-		(fields_autoplaced yes)
-		(effects
-			(font
-				(size 1.27 1.27)
-			)
-			(justify right)
-		)
-		(property "Intersheetrefs" "${INTERSHEET_REFS}"
-			(at 78.8996 119.38 0)
-			(hide yes)
-			(show_name no)
-			(do_not_autoplace no)
-			(effects
-				(font
-					(size 1.27 1.27)
-				)
-				(justify right)
-			)
-		)
-	)
-	(global_label "DDI_B_HPD"
-		(shape input)
-		(at 92.71 156.21 180)
-		(fields_autoplaced yes)
-		(effects
-			(font
-				(size 1.27 1.27)
-			)
-			(justify right)
-		)
-		(property "Intersheetrefs" "${INTERSHEET_REFS}"
-			(at 79.5043 156.21 0)
-			(hide yes)
-			(show_name no)
-			(do_not_autoplace no)
-			(effects
-				(font
-					(size 1.27 1.27)
-				)
-				(justify right)
-			)
-		)
-	)
-	(global_label "DDI_B_TX0-"
-		(shape input)
-		(at 125.73 69.85 180)
-		(fields_autoplaced yes)
-		(effects
-			(font
-				(size 1.27 1.27)
-			)
-			(justify right)
-		)
-		(property "Intersheetrefs" "${INTERSHEET_REFS}"
-			(at 111.4358 69.85 0)
-			(hide yes)
-			(show_name no)
-			(do_not_autoplace no)
-			(effects
-				(font
-					(size 1.27 1.27)
-				)
-				(justify right)
-			)
-		)
-	)
