File: project1/LattepndaCourse/LattepndaCourse.kicad_pcb (KiCad board)
At the start: 2 copper layers, 0 parts

Commit message: Started routing
Parts:
- added A1: LattePanda_Mu, Module_LattePanda:LattePanda_Module_H8.0mm_Horizontal, F.Cu at (398.7, 76.2)
- added BT1: Battery_Cell, A_HDJ_Library:Battery_Holder_CR1220_S8411-45R, F.Cu at (538.0, 238.4)
- added C1: 1uF/16V, A_HDJ_Library:C_0402_1005Metric, F.Cu at (446.5, 98.8)
- added C10: 12pF/50V, A_HDJ_Library:C_0603_1608Metric, F.Cu at (450.0, 86.8)
- added C11: 12pF/50V, A_HDJ_Library:C_0603_1608Metric, F.Cu at (454.1, 71.8)
- added C12: 22uF/10V, A_HDJ_Library:C_0603_1608Metric, F.Cu at (454.1, 74.3)
- added C13: 22uF/10V, A_HDJ_Library:C_0603_1608Metric, F.Cu at (454.1, 76.8)
- added C14: 100nF/10V, A_HDJ_Library:C_0603_1608Metric, F.Cu at (454.1, 79.3)
- added C15: 22uF/10V, A_HDJ_Library:C_0603_1608Metric, F.Cu at (454.1, 81.8)
- added C16: 22uF/10V, A_HDJ_Library:C_0603_1608Metric, F.Cu at (454.1, 84.3)
- added C17: 22uF/10V, A_HDJ_Library:C_0603_1608Metric, F.Cu at (454.1, 86.8)
- added C18: 22uF/10V, A_HDJ_Library:C_0603_1608Metric, F.Cu at (458.1, 71.8)
- added C19: 100nF/10V, A_HDJ_Library:C_0603_1608Metric, F.Cu at (458.1, 74.3)
- added C2: 1uF/16V, A_HDJ_Library:C_0402_1005Metric, F.Cu at (446.5, 100.8)
- added C20: 22uF/10V, A_HDJ_Library:C_0603_1608Metric, F.Cu at (458.1, 76.8)
- added C21: 22uF/10V, A_HDJ_Library:C_0603_1608Metric, F.Cu at (458.1, 79.3)
- added C22: 1uF/16V, A_HDJ_Library:C_0402_1005Metric, F.Cu at (446.5, 104.7)
- added C23: 1uF/16V, A_HDJ_Library:C_0402_1005Metric, F.Cu at (446.5, 106.7)
- added C24: 100nF/50V, A_HDJ_Library:C_0402_1005Metric, F.Cu at (433.8, 175.3)
- added C25: 100nF/50V, A_HDJ_Library:C_0402_1005Metric, F.Cu at (433.8, 177.3)
- added C26: 100nF/50V, A_HDJ_Library:C_0603_1608Metric, F.Cu at (455.3, 124.3)
- added C27: 100nF/50V, A_HDJ_Library:C_0603_1608Metric, F.Cu at (455.3, 126.8)
- added C28: 100nF/50V, A_HDJ_Library:C_0603_1608Metric, F.Cu at (455.3, 129.3)
- added C29: 10uF/10V, A_HDJ_Library:C_0603_1608Metric, F.Cu at (455.3, 131.8)
- added C3: 1uF/16V, A_HDJ_Library:C_0402_1005Metric, F.Cu at (446.5, 102.7)
- added C30: 100nF/50V, A_HDJ_Library:C_0603_1608Metric, F.Cu at (455.3, 134.3)
- added C31: 100uF/25V, A_HDJ_Library:CP_Elec_6.3x7.7, F.Cu at (445.2, 127.1)
- added C32: 560uF/25V, A_HDJ_Library:CP_Elec_6.3x7.7, F.Cu at (445.2, 135.2)
- added C33: 100nF/50V, A_HDJ_Library:C_0402_1005Metric, F.Cu at (463.7, 182.0)
- added C34: 220nF/50V, A_HDJ_Library:C_0402_1005Metric, F.Cu at (451.8, 124.0)
- added C35: 220nF/50V, A_HDJ_Library:C_0402_1005Metric, F.Cu at (451.8, 126.0)
- added C36: 220nF/50V, A_HDJ_Library:C_0402_1005Metric, F.Cu at (451.8, 127.9)
- added C37: 220nF/50V, A_HDJ_Library:C_0402_1005Metric, F.Cu at (451.8, 129.9)
- added C38: 220nF/50V, A_HDJ_Library:C_0402_1005Metric, F.Cu at (451.8, 131.9)
- added C39: 220nF/50V, A_HDJ_Library:C_0402_1005Metric, F.Cu at (451.8, 133.9)
- added C4: 22uF/10V, A_HDJ_Library:C_0603_1608Metric, F.Cu at (450.0, 71.8)
- added C40: 220nF/50V, A_HDJ_Library:C_0402_1005Metric, F.Cu at (451.8, 135.8)
- added C41: 220nF/50V, A_HDJ_Library:C_0402_1005Metric, F.Cu at (451.8, 137.8)
- added C42: 12pF/50V, A_HDJ_Library:C_0402_1005Metric, F.Cu at (463.7, 184.0)
- added C43: 12pF/50V, A_HDJ_Library:C_0402_1005Metric, F.Cu at (463.7, 185.9)
- added C44: 100nF/50V, A_HDJ_Library:C_0402_1005Metric, F.Cu at (463.7, 187.9)
- added C45: 100nF/50V, A_HDJ_Library:C_0402_1005Metric, F.Cu at (466.6, 182.0)
- added C46: 100nF/50V, A_HDJ_Library:C_0402_1005Metric, F.Cu at (466.6, 184.0)
- added C47: 100nF/50V, A_HDJ_Library:C_0402_1005Metric, F.Cu at (466.6, 185.9)
- added C48: 100nF/50V, A_HDJ_Library:C_0402_1005Metric, F.Cu at (466.6, 187.9)
- added C49: 10uF/50V, A_HDJ_Library:C_0402_1005Metric, F.Cu at (469.5, 182.0)
- added C5: 22uF/10V, A_HDJ_Library:C_0603_1608Metric, F.Cu at (450.0, 74.3)
- added C50: 100nF/50V, A_HDJ_Library:C_0402_1005Metric, F.Cu at (469.5, 184.0)
- added C51: 100nF/50V, A_HDJ_Library:C_0402_1005Metric, F.Cu at (469.5, 185.9)
- added C52: 100nF/50V, A_HDJ_Library:C_0402_1005Metric, F.Cu at (469.5, 187.9)
- added C53: 100nF/50V, A_HDJ_Library:C_0402_1005Metric, F.Cu at (472.3, 182.0)
- added C54: 100nF/50V, A_HDJ_Library:C_0402_1005Metric, F.Cu at (472.3, 184.0)
- added C55: 100nF/50V, A_HDJ_Library:C_0402_1005Metric, F.Cu at (472.3, 185.9)
- added C56: 100nF/50V, A_HDJ_Library:C_0402_1005Metric, F.Cu at (472.3, 187.9)
- added C57: 22uF/10V, A_HDJ_Library:C_0603_1608Metric, F.Cu at (381.3, 169.4)
- added C58: 22uF/10V, A_HDJ_Library:C_0603_1608Metric, F.Cu at (381.3, 171.9)
- added C59: 100nF/50V, A_HDJ_Library:C_0603_1608Metric, F.Cu at (381.3, 174.4)
- added C6: 22uF/10V, A_HDJ_Library:C_0603_1608Metric, F.Cu at (450.0, 76.8)
- added C60: 100nF/50V, A_HDJ_Library:C_0603_1608Metric, F.Cu at (381.3, 176.9)
- added C61: 100nF/50V, A_HDJ_Library:C_0603_1608Metric, F.Cu at (381.3, 179.5)
- added C62: 100nF/50V, A_HDJ_Library:C_0603_1608Metric, F.Cu at (381.3, 182.0)
- added C63: 100nF/50V, A_HDJ_Library:C_0603_1608Metric, F.Cu at (458.9, 167.7)
- added C64: 100nF/50V, A_HDJ_Library:C_0603_1608Metric, F.Cu at (458.9, 170.2)
- added C65: 100nF/50V, A_HDJ_Library:C_0603_1608Metric, F.Cu at (458.9, 172.7)
- added C66: 100nF/50V, A_HDJ_Library:C_0603_1608Metric, F.Cu at (458.9, 175.2)
- added C67: 100nF/50V, A_HDJ_Library:C_0603_1608Metric, F.Cu at (458.9, 177.7)
- added C68: 100nF/50V, A_HDJ_Library:C_0603_1608Metric, F.Cu at (462.9, 167.7)
- added C69: 100nF/50V, A_HDJ_Library:C_0603_1608Metric, F.Cu at (462.9, 170.2)
- added C7: 22uF/10V, A_HDJ_Library:C_0603_1608Metric, F.Cu at (450.0, 79.3)
- added C70: 100nF/50V, A_HDJ_Library:C_0603_1608Metric, F.Cu at (462.9, 172.7)
- added C71: 100nF/50V, A_HDJ_Library:C_0603_1608Metric, F.Cu at (462.9, 175.2)
- added C72: 100nF/50V, A_HDJ_Library:C_0603_1608Metric, F.Cu at (394.0, 190.6)
- added C73: 10uF/50V, A_HDJ_Library:C_0603_1608Metric, F.Cu at (394.0, 193.1)
- added C74: 100nF/50V, A_HDJ_Library:C_0603_1608Metric, F.Cu at (394.0, 195.6)
- added C75: 10uF/50V, A_HDJ_Library:C_0603_1608Metric, F.Cu at (394.0, 198.1)
- added C76: 220nF/50V, A_HDJ_Library:C_0603_1608Metric, F.Cu at (398.0, 190.6)
- added C77: 220nF/50V, A_HDJ_Library:C_0603_1608Metric, F.Cu at (398.0, 193.1)
- added C78: 10uF/50V, A_HDJ_Library:C_0603_1608Metric, F.Cu at (398.0, 195.6)
- added C79: 100nF/50V, A_HDJ_Library:C_0603_1608Metric, F.Cu at (398.0, 198.1)
- added C8: 100nF/50V, A_HDJ_Library:C_0603_1608Metric, F.Cu at (450.0, 81.8)
- added C80: 10uF/50V, A_HDJ_Library:C_0603_1608Metric, F.Cu at (402.0, 190.6)
- added C81: 100nF/50V, A_HDJ_Library:C_0603_1608Metric, F.Cu at (402.0, 193.1)
- added C82: 220nF/50V, A_HDJ_Library:C_0603_1608Metric, F.Cu at (402.0, 195.6)
- added C83: 220nF/50V, A_HDJ_Library:C_0603_1608Metric, F.Cu at (402.0, 198.1)
- added C9: 100nF/50V, A_HDJ_Library:C_0603_1608Metric, F.Cu at (450.0, 84.3)
- added D1: ESD9B5.0ST5G, A_HDJ_Library:D_0402_1005Metric, F.Cu at (461.5, 71.5)
- added D10: D_Schottky, A_HDJ_Library:D_SMA, F.Cu at (444.0, 91.0)
- added D11: D_Schottky, A_HDJ_Library:D_SMA, F.Cu at (444.0, 95.5)
- added D12: LED, A_HDJ_Library:LED_0603_1608Metric, F.Cu at (456.4, 103.7)
- added D13: 3V3 lzt=5mA, A_HDJ_Library:D_SOD-323, F.Cu at (473.9, 83.3)
- added D14: LED, A_HDJ_Library:LED_0603_1608Metric, F.Cu at (456.4, 106.3)
- added D15: ESD9B5.0ST5G, A_HDJ_Library:D_0402_1005Metric, F.Cu at (461.5, 81.4)
- added D16: ESD9B5.0ST5G, A_HDJ_Library:D_0402_1005Metric, F.Cu at (461.5, 83.4)
- added D17: 1N5819WS, A_HDJ_Library:D_SOD-323, F.Cu at (430.3, 175.8)
- added D18: 1N5819WS, A_HDJ_Library:D_SOD-323, F.Cu at (430.3, 178.8)
- added D19: ESD9B5.0ST5G, A_HDJ_Library:D_0402_1005Metric, F.Cu at (384.1, 149.6)
- added D2: ESD9B5.0ST5G, A_HDJ_Library:D_0402_1005Metric, F.Cu at (461.5, 73.5)
- added D20: ESD9B5.0ST5G, A_HDJ_Library:D_0402_1005Metric, F.Cu at (384.1, 151.6)
- added D21: ESD9B5.0ST5G, A_HDJ_Library:D_0402_1005Metric, F.Cu at (384.1, 153.6)
- added D22: ESD9B5.0ST5G, A_HDJ_Library:D_0402_1005Metric, F.Cu at (384.1, 155.6)
- added D23: 1N5819WS, A_HDJ_Library:D_SOD-323, F.Cu at (444.4, 172.2)
- added D24: ESD5V0B03, A_HDJ_Library:D_0402_1005Metric, F.Cu at (463.2, 149.6)
- added D25: ESD5V0B03, A_HDJ_Library:D_0402_1005Metric, F.Cu at (463.2, 151.6)
- added D26: ESD5V0B03, A_HDJ_Library:D_0402_1005Metric, F.Cu at (463.2, 153.6)
- added D27: LED_G, A_HDJ_Library:LED_0603_1608Metric, F.Cu at (394.0, 200.7)
- added D3: D_Zener, A_HDJ_Library:D_0402_1005Metric, F.Cu at (461.5, 75.5)
- added D4: D_Zener, A_HDJ_Library:D_0402_1005Metric, F.Cu at (461.5, 77.5)
- added D5: D_Zener, A_HDJ_Library:D_0402_1005Metric, F.Cu at (461.5, 79.5)
- added D6: D_Schottky, A_HDJ_Library:D_SMA, F.Cu at (444.0, 72.8)
- added D7: D_Schottky, A_HDJ_Library:D_SMA, F.Cu at (444.0, 77.3)
- added D8: D_Schottky, A_HDJ_Library:D_SMA, F.Cu at (444.0, 81.9)
- added D9: D_Schottky, A_HDJ_Library:D_SMA, F.Cu at (444.0, 86.4)
- added F1: 6V/1A, A_HDJ_Library:Fuse_0805_2012Metric, F.Cu at (380.4, 150.1)
- added F2: 6V/1A, A_HDJ_Library:Fuse_0805_2012Metric, F.Cu at (380.4, 153.1)
- added F3: 6V/1A, A_HDJ_Library:Fuse_0805_2012Metric, F.Cu at (380.4, 156.0)
- added F4: 6V/1A, A_HDJ_Library:Fuse_0805_2012Metric, F.Cu at (380.4, 159.0)
- added F5: 6V/50mA, A_HDJ_Library:C_0603_1608Metric, F.Cu at (462.9, 177.7)
- added FID1: Fiducial, A_HDJ_Library:Fiducial_0.5mm_Mask1mm, F.Cu at (526.7, 228.8)
- added FID2: Fiducial, A_HDJ_Library:Fiducial_0.5mm_Mask1mm, F.Cu at (526.7, 231.3)
- added H1: MountingHole_Pad, A_HDJ_Library:MountingHole_3.2mm_M3_Pad_Via, F.Cu at (521.5, 231.5)
- added H2: MountingHole_Pad, A_HDJ_Library:MountingHole_3.2mm_M3_Pad_Via, F.Cu at (521.5, 239.4)
- added H3: MountingHole_Pad, A_HDJ_Library:MountingHole_3.2mm_M3_Pad_Via, F.Cu at (521.5, 247.4)
- added H4: MountingHole_Pad, A_HDJ_Library:MountingHole_3.2mm_M3_Pad_Via, F.Cu at (521.5, 255.3)
- added H5: MountingHole_Pad, A_HDJ_Library:MountingHole_3.2mm_M3_Pad_Via, F.Cu at (554.8, 255.4)
- added H6: MountingHole_Pad, A_HDJ_Library:MountingHole_3.2mm_M3_Pad_Via, F.Cu at (554.8, 263.3)
- added H7: MountingHole_Pad, A_HDJ_Library:MountingHole_3mm_M2_Pad_TopOnly, F.Cu at (549.6, 231.1)
- added H8: MountingHole_Pad, A_HDJ_Library:MountingHole_3mm_M2_Pad_TopOnly, F.Cu at (549.6, 238.2)
- added J1: Conn_01x03_Pin, A_HDJ_Library:PinHeader_1x03_P2.54mm_Vertical, F.Cu at (361.8, 139.3)
- added J10: Conn_01x03_Pin, A_HDJ_Library:PinHeader_1x03_P2.54mm_Vertical, F.Cu at (419.3, 151.0)
- added J11: Conn_01x03_Pin, A_HDJ_Library:PinHeader_1x03_P2.54mm_Vertical, F.Cu at (423.9, 151.0)
- added J12: Conn_01x04_Pin, A_HDJ_Library:PinHeader_1x03_P2.54mm_Vertical, F.Cu at (428.6, 151.0)
- added J13: Conn_01x04_Pin, A_HDJ_Library:PinHeader_1x03_P2.54mm_Vertical, F.Cu at (433.2, 151.0)
- added J14: Conn_01x04_Pin, A_HDJ_Library:PinHeader_1x03_P2.54mm_Vertical, F.Cu at (437.9, 151.0)
- added J15: RJ45_RB1-125B8G1A, A_HDJ_Library:RJ45_UDE_RB1-125B8G1A, F.Cu at (446.5, 184.0)
- added J16: Bus_PCI_Express_x4, A_HDJ_Library:PCIe_x4_Gen3Slot_Connectors, F.Cu at (443.6, 115.1)
- added J17: USB_A_Stacked, A_HDJ_Library:USB_A_CUI_UJ2-ADH-TH_Horizontal_Stacked, F.Cu at (373.5, 174.0)
- added J18: USB3_A_Stacked, A_HDJ_Library:USB3_A_Molex_48406-0001_Horizontal_Stacked, F.Cu at (365.3, 155.7)
- added J19: HDMI_A, A_HDJ_Library:HDMI_A_Molex_208658-1001_Horizontal, F.Cu at (447.8, 157.7)
- added J2: USB_C_Receptacle_USB2.0_16P, A_HDJ_Library:USB_C_Receptacle_G-Switch_GT-USB-7010ASV, F.Cu at (542.9, 256.8)
- added J20: Bus_M.2_Socket_M, A_HDJ_Library:PCIe_M.2_Connectors_P=0.5mm_H=4.2mm_KeyM, F.Cu at (401.6, 183.1)
- added J21: Bus_M.2_Socket_E, A_HDJ_Library:PCIe_M.2_Connectors_P=0.5mm_H=4.2mm_KeyE, F.Cu at (392.3, 166.7)
- added J3: Barrel_Jack_Switch, A_HDJ_Library:DC_Jack_DC007B_30V_10A, F.Cu at (454.0, 88.8)
- added J4: Conn_01x04_Pin, A_HDJ_Library:PinHeader_1x03_P2.54mm_Vertical, F.Cu at (391.4, 151.0)
- added J5: Conn_01x04_Pin, A_HDJ_Library:PinHeader_1x03_P2.54mm_Vertical, F.Cu at (396.0, 151.0)
- added J6: Conn_01x04_Pin, A_HDJ_Library:PinHeader_1x03_P2.54mm_Vertical, F.Cu at (400.7, 151.0)
- added J7: Conn_01x04_Pin, A_HDJ_Library:PinHeader_1x03_P2.54mm_Vertical, F.Cu at (405.3, 151.0)
- added J8: Conn_01x03_Pin, A_HDJ_Library:PinHeader_1x03_P2.54mm_Vertical, F.Cu at (410.0, 151.0)
- added J9: Conn_01x03_Pin, A_HDJ_Library:PinHeader_1x03_P2.54mm_Vertical, F.Cu at (414.6, 151.0)
- added JP1: Jumper_3_Bridged12, A_HDJ_Library:PinHeader_1x03_P2.54mm_Vertical, F.Cu at (527.5, 122.5)
- added JP2: NTC_Test, Jumper:SolderJumper-2_P1.3mm_Open_RoundedPad1.0x1.5mm, F.Cu at (418.3, 179.3)
- added L1: 2.2uH/4.3A, A_HDJ_Library:L_Sunlord_SWPA4020S, F.Cu at (474.5, 73.3)
- added L2: 2.2uH/4.3A, A_HDJ_Library:L_Sunlord_SWPA4020S, F.Cu at (474.5, 79.0)
- added M1: Fan_4pin, A_HDJ_Library:JST_PH_B4B-PH-K_1x04_P2.00mm_Vertical, F.Cu at (419.1, 167.1)
- added M2: Fan_4pin, A_HDJ_Library:JST_PH_B4B-PH-K_1x04_P2.00mm_Vertical, F.Cu at (419.1, 173.7)
- added Q1: AON7262E, A_HDJ_Library:MOSFET_PDFN8_3.3x3.3, F.Cu at (451.2, 105.6)
- added Q2: 2N7002H, A_HDJ_Library:SOT-23, F.Cu at (473.5, 90.3)
- added Q3: 2N7002H, A_HDJ_Library:SOT-23, F.Cu at (473.5, 94.7)
- added Q4: 2N7002, A_HDJ_Library:SOT-23, F.Cu at (473.5, 99.2)
- added Q6: 2SK3018, A_HDJ_Library:SOT-23, F.Cu at (459.3, 150.9)
- added Q7: 2SK3018, A_HDJ_Library:SOT-23, F.Cu at (459.3, 155.3)
- added Q8: 2N7002, A_HDJ_Library:SOT-23, F.Cu at (459.3, 159.8)
- added Q9: 2SK3018, A_HDJ_Library:SOT-23, F.Cu at (459.3, 164.2)
- added R1: 10K/1%, A_HDJ_Library:R_0402_1005Metric, F.Cu at (554.6, 228.5)
- added R10: 100K/1%, A_HDJ_Library:R_0402_1005Metric, F.Cu at (464.4, 75.5)
- added R11: 100K/1%, A_HDJ_Library:R_0402_1005Metric, F.Cu at (464.4, 77.5)
- added R12: 10K/1%, A_HDJ_Library:R_0402_1005Metric, F.Cu at (464.4, 79.5)
- added R13: 10K/1%, A_HDJ_Library:R_0402_1005Metric, F.Cu at (464.4, 81.4)
- added R14: 2.5K/1%, A_HDJ_Library:R_0402_1005Metric, F.Cu at (464.4, 83.4)
- added R15: 21.5K/1%, A_HDJ_Library:R_0402_1005Metric, F.Cu at (464.4, 85.4)
- added R16: 21.5K/1%, A_HDJ_Library:R_0402_1005Metric, F.Cu at (467.3, 71.5)
- added R17: 21.5K/1%, A_HDJ_Library:R_0402_1005Metric, F.Cu at (467.3, 73.5)
- added R18: 100K/1%, A_HDJ_Library:R_0402_1005Metric, F.Cu at (467.3, 75.5)
- added R19: 75K/1%, A_HDJ_Library:R_0402_1005Metric, F.Cu at (467.3, 77.5)
- added R2: 10K/1%, A_HDJ_Library:R_0402_1005Metric, F.Cu at (554.6, 230.5)
- added R20: 10K/1%, A_HDJ_Library:R_0402_1005Metric, F.Cu at (467.3, 79.5)
- added R21: 21.5K/1%, A_HDJ_Library:R_0402_1005Metric, F.Cu at (467.3, 81.4)
- added R22: 4.7K/1%, A_HDJ_Library:R_0402_1005Metric, F.Cu at (467.3, 83.4)
- added R23: 2.2K/1%, A_HDJ_Library:R_0402_1005Metric, F.Cu at (467.3, 85.4)
- added R24: 100K/1%, A_HDJ_Library:R_0402_1005Metric, F.Cu at (470.3, 71.5)
- added R25: 100K/1%, A_HDJ_Library:R_0402_1005Metric, F.Cu at (470.3, 73.5)
- added R26: 10K/1%, A_HDJ_Library:R_0402_1005Metric, F.Cu at (470.3, 75.5)
- added R27: 2.2K/1%, A_HDJ_Library:R_0402_1005Metric, F.Cu at (470.3, 77.5)
- added R28: 100R/1%, A_HDJ_Library:R_0402_1005Metric, F.Cu at (470.3, 79.5)
- added R29: 100R/1%, A_HDJ_Library:R_0402_1005Metric, F.Cu at (470.3, 81.4)
- added R3: 10K/1%, A_HDJ_Library:R_0402_1005Metric, F.Cu at (554.6, 232.5)
- added R30: 100R/1%, A_HDJ_Library:R_0402_1005Metric, F.Cu at (470.3, 83.4)
- added R31: 100R/1%, A_HDJ_Library:R_0402_1005Metric, F.Cu at (470.3, 85.4)
- added R32: 4.7K/1%, A_HDJ_Library:R_0402_1005Metric, F.Cu at (429.5, 165.4)
- added R33: 21.5K/1%, A_HDJ_Library:R_0402_1005Metric, F.Cu at (429.5, 167.4)
- added R34: 100R/1%, A_HDJ_Library:R_0402_1005Metric, F.Cu at (429.5, 169.4)
- added R35: 21.5K/1%, A_HDJ_Library:R_0402_1005Metric, F.Cu at (429.5, 171.4)
- added R36: 100R/1%, A_HDJ_Library:R_0402_1005Metric, F.Cu at (429.5, 173.4)
- added R37: 4.7K/1%, A_HDJ_Library:R_0402_1005Metric, F.Cu at (432.5, 165.4)
- added R38: 4.7K/1%, A_HDJ_Library:R_0402_1005Metric, F.Cu at (432.5, 167.4)
- added R39: 21.5K/1%, A_HDJ_Library:R_0402_1005Metric, F.Cu at (432.5, 169.4)
- added R4: 100K/1%, A_HDJ_Library:R_0402_1005Metric, F.Cu at (554.6, 234.5)
- added R40: 4.7K/1%, A_HDJ_Library:R_0402_1005Metric, F.Cu at (432.5, 171.4)
- added R41: 21.5K/1%, A_HDJ_Library:R_0402_1005Metric, F.Cu at (432.5, 173.4)
- added R42: 0R/1%, A_HDJ_Library:R_0402_1005Metric, F.Cu at (435.4, 165.4)
- added R43: 0R/1%, A_HDJ_Library:R_0402_1005Metric, F.Cu at (435.4, 167.4)
- added R44: 10K/1%, A_HDJ_Library:R_0402_1005Metric, F.Cu at (435.4, 169.4)
- added R45: 470R/1%, A_HDJ_Library:R_0402_1005Metric, F.Cu at (463.7, 189.9)
- added R46: 470R/1%, A_HDJ_Library:R_0402_1005Metric, F.Cu at (463.7, 191.9)
- added R47: 1M/1%, A_HDJ_Library:R_0402_1005Metric, F.Cu at (463.7, 193.9)
- added R48: 2.49K/1%, A_HDJ_Library:R_0603_1608Metric, F.Cu at (467.2, 200.4)
- added R49: 10K/1%, A_HDJ_Library:R_0402_1005Metric, F.Cu at (463.7, 195.8)
- added R5: 100K/1%, A_HDJ_Library:R_0402_1005Metric, F.Cu at (554.6, 236.5)
- added R50: 10K/1%, A_HDJ_Library:R_0402_1005Metric, F.Cu at (463.7, 197.8)
- added R51: 470R/1%, A_HDJ_Library:R_0402_1005Metric, F.Cu at (463.2, 155.6)
- added R52: 470R/1%, A_HDJ_Library:R_0402_1005Metric, F.Cu at (463.2, 157.6)
- added R53: 470R/1%, A_HDJ_Library:R_0402_1005Metric, F.Cu at (463.2, 159.6)
- added R54: 470R/1%, A_HDJ_Library:R_0402_1005Metric, F.Cu at (463.2, 161.6)
- added R55: 470R/1%, A_HDJ_Library:R_0402_1005Metric, F.Cu at (466.1, 149.6)
- added R56: 470R/1%, A_HDJ_Library:R_0402_1005Metric, F.Cu at (466.1, 151.6)
- added R57: 470R/1%, A_HDJ_Library:R_0402_1005Metric, F.Cu at (466.1, 153.6)
- added R58: 470R/1%, A_HDJ_Library:R_0402_1005Metric, F.Cu at (466.1, 155.6)
- added R59: 2.5K/1%, A_HDJ_Library:R_0402_1005Metric, F.Cu at (466.1, 157.6)
- added R6: 1K/1%, A_HDJ_Library:R_0402_1005Metric, F.Cu at (554.6, 238.4)
- added R60: 2.2K/1%, A_HDJ_Library:R_0402_1005Metric, F.Cu at (466.1, 159.6)
- added R61: 2.2K/1%, A_HDJ_Library:R_0402_1005Metric, F.Cu at (466.1, 161.6)
- added R62: 2.2K/1%, A_HDJ_Library:R_0402_1005Metric, F.Cu at (469.0, 149.6)
- added R63: 2.2K/1%, A_HDJ_Library:R_0402_1005Metric, F.Cu at (469.0, 151.6)
- added R64: 1M/1%, A_HDJ_Library:R_0402_1005Metric, F.Cu at (469.0, 153.6)
- added R65: 0R/1%, A_HDJ_Library:R_0402_1005Metric, F.Cu at (390.5, 190.3)
- added R66: 1K/1%, A_HDJ_Library:R_0402_1005Metric, F.Cu at (469.0, 155.6)
- added R67: 21.5K/1%, A_HDJ_Library:R_0402_1005Metric, F.Cu at (469.0, 157.6)
- added R68: 0R/1%, A_HDJ_Library:R_0402_1005Metric, F.Cu at (390.5, 192.3)
- added R69: 0R/1%, A_HDJ_Library:R_0402_1005Metric, F.Cu at (390.5, 194.3)
- added R7: 1K/1%, A_HDJ_Library:R_0402_1005Metric, F.Cu at (461.5, 85.4)
- added R70: 0R/1%, A_HDJ_Library:R_0402_1005Metric, F.Cu at (390.5, 196.3)
- added R71: 0R/1%, A_HDJ_Library:R_0402_1005Metric, F.Cu at (390.5, 198.3)
- added R72: 10K/1%, A_HDJ_Library:R_0402_1005Metric, F.Cu at (390.5, 200.3)
- added R73: 10K/1%, A_HDJ_Library:R_0402_1005Metric, F.Cu at (390.5, 202.3)
- added R8: 10K/1%, A_HDJ_Library:R_0402_1005Metric, F.Cu at (464.4, 71.5)
- added R9: 56K/1%, A_HDJ_Library:R_0402_1005Metric, F.Cu at (464.4, 73.5)
- added SW1: SW_Push, A_HDJ_Library:SW_Push_6x6x6, F.Cu at (465.5, 91.6)
- added SW2: SW_Push, A_HDJ_Library:SW_Push_6x6x6, F.Cu at (465.5, 98.7)
- added TH1: NTC-10K, A_HDJ_Library:R_0603_1608Metric, F.Cu at (422.5, 178.8)
- added TP1: TestPoint, A_HDJ_Library:TestPoint_Pad_D1.5mm, F.Cu at (547.8, 243.6)
- added TP10: TestPoint, A_HDJ_Library:TestPoint_Pad_D1.5mm, F.Cu at (559.8, 232.8)
- added TP11: TestPoint, A_HDJ_Library:TestPoint_Pad_D1.5mm, F.Cu at (559.8, 236.4)
- added TP12: TestPoint, A_HDJ_Library:TestPoint_Pad_D1.5mm, F.Cu at (559.8, 239.9)
- added TP13: TestPoint, A_HDJ_Library:TestPoint_Pad_D1.5mm, F.Cu at (559.8, 245.5)
- added TP14: TestPoint, A_HDJ_Library:TestPoint_Pad_D1.5mm, F.Cu at (560.5, 253.2)
- added TP2: TestPoint, A_HDJ_Library:TestPoint_Pad_D1.5mm, F.Cu at (531.8, 253.2)
- added TP3: TestPoint, A_HDJ_Library:TestPoint_Pad_D1.5mm, F.Cu at (531.8, 256.7)
- added TP4: TestPoint, A_HDJ_Library:TestPoint_Pad_D1.5mm, F.Cu at (531.8, 260.3)
- added TP5: TestPoint, A_HDJ_Library:TestPoint_Pad_D1.5mm, F.Cu at (531.8, 263.8)
- added TP6: TestPoint, A_HDJ_Library:TestPoint_Pad_D1.5mm, F.Cu at (535.3, 253.2)
- added TP7: TestPoint, A_HDJ_Library:TestPoint_Pad_D1.5mm, F.Cu at (535.3, 256.7)
- added TP8: TestPoint, A_HDJ_Library:TestPoint_Pad_D1.5mm, F.Cu at (535.3, 260.3)
- added TP9: TestPoint, A_HDJ_Library:TestPoint_Pad_D1.5mm, F.Cu at (559.8, 229.3)
- added U1: USB PD等快充协议受电芯片-CH224K-ESSOP10, A_HDJ_Library:ESSOP-10-1EP_3.9x5mm_P1.0mm_EP3.2x2.3, F.Cu at (463.9, 105.8)
- added U10: RTL8111H-CG-RH, A_HDJ_Library:QFN-32-1EP_4x4mm_P0.4mm_EP2.65x2.65mm, F.Cu at (468.3, 192.0)
- added U11: ULC0524P, A_HDJ_Library:Diodes_UDFN-10_1.0x2.5mm_P0.5mm, F.Cu at (466.7, 197.2)
- added U12: ULC0524P, A_HDJ_Library:Diodes_UDFN-10_1.0x2.5mm_P0.5mm, F.Cu at (469.6, 197.2)
- added U13: ULC0524P, A_HDJ_Library:Diodes_UDFN-10_1.0x2.5mm_P0.5mm, F.Cu at (379.7, 162.5)
- added U14: ULC0524P, A_HDJ_Library:Diodes_UDFN-10_1.0x2.5mm_P0.5mm, F.Cu at (382.6, 162.5)
- added U15: ULC0524P, A_HDJ_Library:Diodes_UDFN-10_1.0x2.5mm_P0.5mm, F.Cu at (385.6, 162.5)
- added U16: ULC0524P, A_HDJ_Library:Diodes_UDFN-10_1.0x2.5mm_P0.5mm, F.Cu at (443.7, 168.7)
- added U17: ULC0524P, A_HDJ_Library:Diodes_UDFN-10_1.0x2.5mm_P0.5mm, F.Cu at (446.6, 168.7)
- added U2: TL431D, A_HDJ_Library:SOT-23, F.Cu at (473.5, 103.6)
- added U3: LM2734X, A_HDJ_Library:TSOT-23-6, F.Cu at (442.5, 100.1)
- added U4: LM2734X, A_HDJ_Library:TSOT-23-6, F.Cu at (442.5, 104.6)
- added U5: ULC0524P, A_HDJ_Library:Diodes_UDFN-10_1.0x2.5mm_P0.5mm, F.Cu at (390.5, 160.4)
- added U6: ULC0524P, A_HDJ_Library:Diodes_UDFN-10_1.0x2.5mm_P0.5mm, F.Cu at (393.5, 160.4)
- added U7: ULC0524P, A_HDJ_Library:Diodes_UDFN-10_1.0x2.5mm_P0.5mm, F.Cu at (396.4, 160.4)
- added U8: ULC0524P, A_HDJ_Library:Diodes_UDFN-10_1.0x2.5mm_P0.5mm, F.Cu at (399.4, 160.4)
- added U9: ULC0524P, A_HDJ_Library:Diodes_UDFN-10_1.0x2.5mm_P0.5mm, F.Cu at (402.3, 160.4)
- added Y1: 25MHz, A_HDJ_Library:Crystal_SMD_3225-4Pin_3.2x2.5mm, F.Cu at (520.1, 263.5)
Other:
- board outline added: 165 x 84 mm
- copper layers 2 -> 4
