File: project1/LattepndaCourse/PCIe.kicad_sch (KiCad schematic)
At the start: 0 parts

Commit message: Hierachi
Other:
- title: (none) -> practice design
Changed lines of the file:
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@@
 	(generator "eeschema")
 	(generator_version "9.0")
-	(paper "A4")
+	(paper "A2")
+	(title_block
+		(title "practice design")
+		(date "2026-09-30")
+		(rev "1")
+	)
 )

Commit message: PCIe is done
Parts:
- added C26, C27, C28, C30: 100nF/50V, A_HDJ_Library:C_0603_1608Metric, symbol Device:C_Small
- added C29: 10uF/10V, A_HDJ_Library:C_0603_1608Metric, symbol Device:C_Small
- added C31: 100uF/25V, A_HDJ_Library:CP_Elec_6.3x7.7, symbol Device:C_Polarized
- added C32: 560uF/25V, A_HDJ_Library:CP_Elec_6.3x7.7, symbol Device:C_Polarized
- added C34, C35, C36, C37, C38, C39, C40, C41: 220nF/50V, A_HDJ_Library:C_0402_1005Metric, symbol Device:C_Small
- added J16: Bus_PCI_Express_x4, A_HDJ_Library:PCIe_x4_Gen3Slot_Connectors, symbol Connector:Bus_PCI_Express_x4
- added TP13: TestPoint, symbol Connector:TestPoint
Connections:
- new net: C26.2, C27.2, C31.1, J16.A2 (+12V), J16.A3 (+12V), J16.B1 (+12V), J16.B2 (+12V), J16.B3 (+12V)
- new net +3.3V: C28.1, C29.1, C30.2, C32.1, J16.A10 (+3.3V), J16.A9 (+3.3V), J16.B10 (3.3Vaux), J16.B8 (+3.3V)
- new net GND: C26.1, C27.1, C28.2, C29.2, C30.1, C31.2, C32.2, J16.A1 (~{PRSNT1}), J16.A12 (GND), J16.A15 (GND), J16.A18 (GND), J16.A20 (GND), J16.A23 (GND), J16.A24 (GND), J16.A27 (GND), J16.A28 (GND), J16.A31 (GND), J16.A4 (GND), J16.B13 (GND), J16.B16 (GND), J16.B17 (~{PRSNT2}), J16.B18 (GND), J16.B21 (GND), J16.B22 (GND), J16.B25 (GND), J16.B26 (GND), J16.B29 (GND), J16.B31 (~{PRSNT2}), J16.B32 (GND), J16.B4 (GND), J16.B7 (GND)
- new net PCIE30_TX0_N: C35.2, J16.B15 (PETn0)
- new net PCIE30_TX0_P: C34.2, J16.B14 (PETp0)
- new net PCIE30_TX1_N: C37.2, J16.B20 (PETn1)
- new net PCIE30_TX1_P: C36.2, J16.B19 (PETp1)
- new net PCIE30_TX2_N: C39.2, J16.B24 (PETn2)
- new net PCIE30_TX2_P: C38.2, J16.B23 (PETp2)
- new net PCIE30_TX3_N: C41.2, J16.B28 (PETn3)
- new net PCIE30_TX3_P: C40.2, J16.B27 (PETp3)
- new net PCIE_RX_0+: J16.A16 (PERp0)
- new net PCIE_RX_0-: J16.A17 (PERn0)
- new net PCIE_RX_1+: J16.A21 (PERp1)
- new net PCIE_RX_1-: J16.A22 (PERn1)
- new net PCIE_RX_2+: J16.A25 (PERp2)
- new net PCIE_RX_2-: J16.A26 (PERn2)
- new net PCIE_RX_3+: J16.A29 (PERp3)
- new net PCIE_RX_3-: J16.A30 (PERn3)
- new net PCIE_TX_0+: C34.1
- new net PCIE_TX_0-: C35.1
- new net PCIE_TX_1+: C36.1
- new net PCIE_TX_1-: C37.1
- new net PCIE_TX_2+: C38.1
- new net PCIE_TX_2-: C39.1
- new net PCIE_TX_3+: C40.1
- new net PCIE_TX_3-: C41.1
- new net PE_RST: J16.A11 (~{PERST}), TP13.1
- new net REFCLK+: J16.A13 (REFCLK+)
- new net REFCLK-: J16.A14 (REFCLK-)
- new net ~{WAKE}: J16.B11 (~{WAKE})
- no-connect marks 0 -> 11

Commit message: USB is done
Connections:
- net +12V: now reaches C26.2, C27.2, C31.1, J16.A2 (+12V), J16.A3 (+12V), J16.B1 (+12V), J16.B2 (+12V), J16.B3 (+12V)
Changed lines of the file:
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@@
+	)
+	(junction
+		(at 133.35 62.23)
+		(diameter 0)
+		(color 0 0 0 0)
 	)
 	(junction
@@
 	(wire
 		(pts
+			(xy 133.35 62.23) (xy 128.27 62.23)
+		)
+		(stroke
+			(width 0)
+			(type default)
+		)
+	)
+	(wire
+		(pts
 			(xy 163.83 116.84) (xy 185.42 116.84)
 		)
@@
 	(wire
 		(pts
+			(xy 133.35 59.69) (xy 133.35 62.23)
+		)
+		(stroke
+			(width 0)
+			(type default)
+		)
+	)
+	(wire
+		(pts
 			(xy 127 104.14) (xy 133.35 104.14)
 		)
@@
 	(wire
 		(pts
-			(xy 146.05 62.23) (xy 128.27 62.23)
+			(xy 146.05 62.23) (xy 133.35 62.23)
 		)
 		(stroke
@@
 					(unit 1)
 				)
+			)
+		)
+	)
+	(symbol
+		(lib_id "power:+12V")
+		(at 133.35 59.69 0)
+		(unit 1)
+		(body_style 1)
+		(exclude_from_sim no)
+		(in_bom yes)
+		(on_board yes)
+		(in_pos_files yes)
+		(dnp no)
+		(fields_autoplaced yes)
+		(property "Reference" "#PWR092"
+			(at 133.35 63.5 0)
+			(hide yes)
+			(show_name no)
+			(do_not_autoplace no)
+			(effects
+				(font
+					(size 1.27 1.27)
+				)
+			)
+		)
+		(property "Value" "+12V"
+			(at 133.35 54.61 0)
+			(show_name no)
+			(do_not_autoplace no)
+			(effects
+				(font
+					(size 1.27 1.27)
+				)
+			)
+		)
+		(property "Footprint" ""
+			(at 133.35 59.69 0)
+			(hide yes)
+			(show_name no)
+			(do_not_autoplace no)
+			(effects
+				(font
+					(size 1.27 1.27)
+				)
+			)
+		)
+		(property "Datasheet" ""
+			(at 133.35 59.69 0)
+			(hide yes)
+			(show_name no)
+			(do_not_autoplace no)
+			(effects
+				(font
+					(size 1.27 1.27)
+				)
+			)
+		)
+		(property "Description" "Power symbol creates a global label with name \"+12V\""
+			(at 133.35 59.69 0)
+			(hide yes)
+			(show_name no)
+			(do_not_autoplace no)
+			(effects
+				(font
+					(size 1.27 1.27)
+				)
+			)
+		)
+		(pin "1"
+		)
+		(instances
+			(project "LattepndaCourse"
+				(path "/4e04f3a7-ba43-4db9-8bbc-1a27efcf5abf/71be7a07-db75-4263-ad02-00a7dbc381e2"
+					(reference "#PWR092")
+					(unit 1)
+				)

Commit message: Hierachi needs some work
Parts:
- C26, C27, C28, C29, C30, C31, C32, C34, C35, C36, C37, C38, C39, C40, C41, J16, TP13: now not fitted
Connections:
- net +12V renamed +12VA

Commit message: Started routing
Parts:
- TP13: footprint (none) -> A_HDJ_Library:TestPoint_Pad_D1.5mm
