File: project1/LattepndaCourse/PowerSupply.kicad_sch (KiCad schematic)
At the start: 0 parts

Commit message: Hierachi
Other:
- title: (none) -> practice design
Changed lines of the file:
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@@
 	(generator "eeschema")
 	(generator_version "9.0")
-	(paper "A4")
+	(paper "A2")
+	(title_block
+		(title "practice design")
+		(date "2026-09-30")
+		(rev "1")
+	)
 )

Commit message: Up to power jack
Parts:
- added C1: 1uF/16V, A_HDJ_Library:C_0402_1005Metric, symbol Device:C_Small
- added D1, D2: ESD9B5.0ST5G, A_HDJ_Library:D_0402_1005Metric, symbol Diode:ESD9B5.0ST5G
- added D10, D11, D6, D7, D8, D9: D_Schottky, A_HDJ_Library:D_SMA, symbol Device:D_Schottky
- added D3, D4, D5: D_Zener, A_HDJ_Library:D_0402_1005Metric, symbol Device:D_Zener
- added J2: USB_C_Receptacle_USB2.0_16P, symbol Connector:USB_C_Receptacle_USB2.0_16P
- added J3: Barrel_Jack_Switch, A_HDJ_Library:DC_Jack_DC007B_30V_10A, symbol Connector:Barrel_Jack_Switch
- added R7: 1K/1%, A_HDJ_Library:R_0402_1005Metric, symbol Device:R
- added R8: 10K/1%, A_HDJ_Library:R_0402_1005Metric, symbol Device:R
- added R9: 56K/1%, A_HDJ_Library:R_0402_1005Metric, symbol Device:R
- added TP2, TP3, TP4: TestPoint, symbol Connector:TestPoint
- added U1: USB PD等快充协议受电芯片-CH224K-ESSOP10, A_HDJ_Library:ESSOP-10-1EP_3.9x5mm_P1.0mm_EP3.2x2.3, symbol A_HDJ_Library:CH224K
Connections:
- new net: D10.1 (K), D11.1 (K), D6.1 (K), D7.1 (K), D8.1 (K), D9.1 (K), TP4.1
- new net: C1.1, R7.2, U1.1 (VDD)
- new net: R8.2, U1.8 (VBUS)
- new net: R9.1, U1.9 (CFG1)
- new net +12V: D6.2 (A), D7.2 (A), D8.2 (A), J3.1, TP2.1
- new net +15V: D10.2 (A), D11.2 (A), D3.1 (K), D9.2 (A), J2.A4 (VBUS), J2.A9 (VBUS), J2.B4 (VBUS), J2.B9 (VBUS), R7.1, R8.1, TP3.1
- new net CC1: D4.1 (K), J2.A5 (CC1), U1.7 (CC1)
- new net CC2: D5.1 (K), J2.B5 (CC2), U1.6 (CC2)
- new net GND: C1.2, D1.1 (A1), D2.1 (A1), D3.2 (A), D4.2 (A), D5.2 (A), J2.A1 (GND), J2.A12 (GND), J2.B1 (GND), J2.B12 (GND), J2.SH (SHIELD), J3.2, J3.3, R9.2, U1.0 (GND)
- new net PWR_C_D+: D2.2 (A2), J2.A6 (D+), J2.B6 (D+), U1.4 (DP)
- new net PWR_C_D-: D1.2 (A2), J2.A7 (D-), J2.B7 (D-), U1.5 (DM)
- no-connect marks 0 -> 5
Other:
- note added: "CH224K get DC 15V power from USB-PD adapter"

Commit message: still working on power
Parts:
- added C10, C11: 12pF/50V, A_HDJ_Library:C_0603_1608Metric, symbol Device:C_Small
- added C12, C13, C15, C16, C17, C18, C20, C21, C4, C5, C6, C7: 22uF/10V, A_HDJ_Library:C_0603_1608Metric, symbol Device:C_Small
- added C14, C19: 100nF/10V, A_HDJ_Library:C_0603_1608Metric, symbol Device:C_Small
- added C2, C3: 1uF/16V, A_HDJ_Library:C_0402_1005Metric, symbol Device:C_Small
- added C8, C9: 100nF/50V, A_HDJ_Library:C_0603_1608Metric, symbol Device:C_Small
- added D12: LED, A_HDJ_Library:LED_0603_1608Metric, symbol Device:LED
- added D13: 3V3 lzt=5mA, A_HDJ_Library:D_SOD-323, symbol Device:D_Schottky
- added L1, L2: 2.2uH/4.3A, A_HDJ_Library:L_Sunlord_SWPA4020S, symbol Device:L
- added Q1: AON7262E, A_HDJ_Library:MOSFET_PDFN8_3.3x3.3, symbol A_HDJ_Library:AON7262E
- added Q2, Q3: 2N7002H, A_HDJ_Library:SOT-23, symbol Transistor_FET:2N7002H
- added R10, R11, R18: 100K/1%, A_HDJ_Library:R_0402_1005Metric, symbol Device:R
- added R12, R13, R20: 10K/1%, A_HDJ_Library:R_0402_1005Metric, symbol Device:R
- added R14: 2.5K/1%, A_HDJ_Library:R_0402_1005Metric, symbol Device:R
- added R15, R16, R17, R21: 21.5K/1%, A_HDJ_Library:R_0402_1005Metric, symbol Device:R
- added R19: 75K/1%, A_HDJ_Library:R_0402_1005Metric, symbol Device:R
- added R22: 4.7K/1%, A_HDJ_Library:R_0402_1005Metric, symbol Device:R
- added R23: 2.2K/1%, A_HDJ_Library:R_0402_1005Metric, symbol Device:R
- added TP5, TP6, TP7, TP8: TestPoint, symbol Connector:TestPoint
- added U2: TL431D, A_HDJ_Library:SOT-23, symbol Reference_Voltage:TL431D
- added U3, U4: LM2734X, A_HDJ_Library:TSOT-23-6, symbol Regulator_Switching:LM2734X
Connections:
- net +12V: now also C2.2, Q1.1 (S_1), Q1.10 (D_6), Q1.11 (D_7), Q1.2 (S_2), Q1.3 (S_3), Q1.5 (D_1), Q1.6 (D_2), Q1.7 (D_3), Q1.8 (D_4), Q1.9 (D_5), R10.1, R12.2, R13.2, R17.1, TP5.1
- net GND: now also C3.2, C4.2, C5.1, C6.2, C7.1, D12.1 (K), D13.2 (A), Q3.2 (S), R14.1, R16.2, R18.1, R20.1, R22.1, U2.2 (A), U2.3 (A), U2.6 (A), U2.7 (A), U3.2 (GND), U4.2 (GND)
- net VDC: now reaches D10.1 (K), D11.1 (K), D6.1 (K), D7.1 (K), D8.1 (K), D9.1 (K), TP4.1
- net VDC: now also C4.1, C5.2, C6.1, C7.2, R23.2, U3.5 (VIN), U4.5 (VIN)
- new net: C2.1, Q1.4 (G), R10.2, R11.2
- new net: D12.2 (A), R17.2
- new net: C8.1, U4.1 (BOOST)
- new net: C8.2, L2.1, U4.6 (SW)
- new net: C3.1, Q2.1 (G), Q3.1 (G), R15.1, R16.1
- new net: Q2.2 (S), Q3.3 (D)
- new net: C11.1, C17.1, C18.1, C19.1, C20.1, C21.1, R21.1, R22.2, U4.3 (FB)
- new net: R13.1, R14.2, U2.8 (REF)
- new net: C10.1, C12.1, C13.1, C14.1, C15.1, C16.1, R19.1, R20.2, U3.3 (FB)
- new net: R12.1, R15.2, U2.1 (K)
- new net: Q2.3 (D), R11.1
- new net: C9.1, U3.1 (BOOST)
- new net: C9.2, L1.1, U3.6 (SW)
- new net +3.3V: C11.2, C17.2, C18.2, C19.2, C20.2, C21.2, L2.2, R21.2, TP7.1
- new net +5V: C10.2, C12.2, C13.2, C14.2, C15.2, C16.2, L1.2, R19.2, TP6.1
- new net PWR_EN: R18.2, U3.4 (EN), U4.4 (EN)
- new net PullUp: D13.1 (K), R23.1, TP8.1
Other:
- note added: "For soft start"
- note added: "PCIe power enable LED"
- note added: "Power for PCIe x4 OVP813.86V"
- note added: "Pullup power for bios_sel"

Commit message: power is done
Parts:
- added C22, C23: 1uF/16V, A_HDJ_Library:C_0402_1005Metric, symbol Device:C_Small
- added D14: LED, A_HDJ_Library:LED_0603_1608Metric, symbol Device:LED
- added D15, D16: ESD9B5.0ST5G, A_HDJ_Library:D_0402_1005Metric, symbol Diode:ESD9B5.0ST5G
- added JP1: Jumper_3_Bridged12, symbol Jumper:Jumper_3_Bridged12
- added Q4: 2N7002, A_HDJ_Library:SOT-23, symbol Transistor_FET:2N7002
- added R24, R25: 100K/1%, A_HDJ_Library:R_0402_1005Metric, symbol Device:R
- added R26: 10K/1%, A_HDJ_Library:R_0402_1005Metric, symbol Device:R
- added R27: 2.2K/1%, A_HDJ_Library:R_0402_1005Metric, symbol Device:R
- added R28, R29, R30, R31: 100R/1%, A_HDJ_Library:R_0402_1005Metric, symbol Device:R
- added SW1, SW2: SW_Push, A_HDJ_Library:SW_Push_6x6x6, symbol Switch:SW_Push
Connections:
- net +3.3V: now also R27.2
- net GND: now also C22.1, C23.1, D15.2 (A2), D16.2 (A2), Q4.2 (S), R26.1, SW1.2, SW2.2
- net PWR_EN: now also R24.1
- new net: C22.2, D15.1 (A1), R28.2, R29.1, SW1.1
- new net: C23.2, D16.1 (A1), R30.2, R31.1, SW2.1
- new net: Q4.1 (G), R25.1, R26.2
- new net: D14.1 (K), Q4.3 (D)
- new net: JP1.2 (C), R24.2
- new net: D14.2 (A), R27.1
- new net +3V3: R29.2, R31.2
- new net SLS_S3: JP1.3 (B)
- new net ~{PWR_LED}/~{PSON}: JP1.1 (A), R25.2
- new net ~{PWR_SW}: R28.1
- new net ~{RST_SW}: R30.1
Other:
- note added: ".SY8253ADC 23V 3A 500kHz"
- note added: "12V DC Input(12V 6A-10A)"
- note added: "15V PD Input"
- note added: "LattePanda has Pull-Up resistors"
- note added: "Vout = 0.6*(21.5 + 4.7)/4.7 = 3.446V"
- note added: "Vout = 0.6*(75 + 10)/10 = 5.1V"
- moved on the sheet: C1, C10, C11, C12, C13, C14, C15, C16, C17, C18, C19, C2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

Commit message: USB is done
Changed lines of the file:
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@@
 	)
 	(junction
+		(at 105.41 143.51)
+		(diameter 0)
+		(color 0 0 0 0)
+	)
+	(junction
 		(at 515.62 190.5)
 		(diameter 0)
@@
 	)
 	(junction
-		(at 105.41 143.51)
-		(diameter 0)
-		(color 0 0 0 0)
-	)
-	(junction
 		(at 506.73 151.13)
 		(diameter 0)
@@
 	)
 	(junction
-		(at 105.41 140.97)
-		(diameter 0)
-		(color 0 0 0 0)
-	)
-	(junction
 		(at 289.56 66.04)
 		(diameter 0)
@@
 	(wire
 		(pts
-			(xy 105.41 143.51) (xy 105.41 147.32)
-		)
-		(stroke
-			(width 0)
-			(type default)
-		)
-	)
-	(wire
-		(pts
 			(xy 219.71 90.17) (xy 219.71 110.49)
 		)
@@
 	)
 	(symbol
-		(lib_id "power:GND")
-		(at 105.41 147.32 0)
-		(unit 1)
-		(body_style 1)
-		(exclude_from_sim no)
-		(in_bom yes)
-		(on_board yes)
-		(in_pos_files yes)
-		(dnp no)
-		(fields_autoplaced yes)
-		(property "Reference" "#PWR021"
-			(at 105.41 153.67 0)
-			(hide yes)
-			(show_name no)
-			(do_not_autoplace no)
-			(effects
-				(font
-					(size 1.27 1.27)
-				)
-			)
-		)
-		(property "Value" "GND"
-			(at 105.41 152.4 0)
-			(show_name no)
-			(do_not_autoplace no)
-			(effects
-				(font
-					(size 1.27 1.27)
-				)
-			)
-		)
-		(property "Footprint" ""
-			(at 105.41 147.32 0)
-			(hide yes)
-			(show_name no)
-			(do_not_autoplace no)
-			(effects
-				(font
-					(size 1.27 1.27)
-				)
-			)
-		)
-		(property "Datasheet" ""
-			(at 105.41 147.32 0)
-			(hide yes)
-			(show_name no)
-			(do_not_autoplace no)
-			(effects
-				(font
-					(size 1.27 1.27)
-				)
-			)
-		)
-		(property "Description" "Power symbol creates a global label with name \"GND\" , ground"
-			(at 105.41 147.32 0)
-			(hide yes)
-			(show_name no)
-			(do_not_autoplace no)
-			(effects
-				(font
-					(size 1.27 1.27)
-				)
-			)
-		)
-		(pin "1"
-		)
-		(instances
-			(project "LattepndaCourse"
-				(path "/4e04f3a7-ba43-4db9-8bbc-1a27efcf5abf/dc3c01ed-4c1a-4ffc-b57d-00aa66dee251"
-					(reference "#PWR021")
-					(unit 1)
-				)
-			)
-		)
-	)
-	(symbol
 		(lib_id "Transistor_FET:2N7002")
 		(at 334.01 217.17 0)
@@
 	)
 	(symbol
-		(lib_id "Device:R")
-		(at 320.04 118.11 270)
+		(lib_id "power:GND")
+		(at 105.41 143.51 0)
 		(unit 1)
 		(body_style 1)
@@
 		(in_pos_files yes)
 		(dnp no)
-		(property "Reference" "R23"
-			(at 319.786 115.824 90)
+		(fields_autoplaced yes)
+		(property "Reference" "#PWR021"
+			(at 105.41 149.86 0)
+			(hide yes)
 			(show_name no)
 			(do_not_autoplace no)
@@
 			)
 		)
-		(property "Value" "2.2K/1%"
-			(at 318.008 120.396 90)
+		(property "Value" "GND"
+			(at 105.41 148.59 0)
 			(show_name no)
 			(do_not_autoplace no)
@@
 			)
 		)
-		(property "Footprint" "A_HDJ_Library:R_0402_1005Metric"
-			(at 320.04 116.332 90)
+		(property "Footprint" ""
+			(at 105.41 143.51 0)
 			(hide yes)
 			(show_name no)
@@
 		)
 		(property "Datasheet" ""
-			(at 320.04 118.11 0)
+			(at 105.41 143.51 0)
 			(hide yes)
 			(show_name no)
@@
 			)
 		)
-		(property "Description" "Resistor"
-			(at 320.04 118.11 0)
+		(property "Description" "Power symbol creates a global label with name \"GND\" , ground"
+			(at 105.41 143.51 0)
 			(hide yes)
 			(show_name no)
@@
 			)
 		)
-		(pin "2"
-		)
 		(pin "1"
 		)
@@
 			(project "LattepndaCourse"
 				(path "/4e04f3a7-ba43-4db9-8bbc-1a27efcf5abf/dc3c01ed-4c1a-4ffc-b57d-00aa66dee251"
-					(reference "R23")
+					(reference "#PWR021")
 					(unit 1)
 				)
@@
 	)
 	(symbol
-		(lib_id "Connector:TestPoint")
-		(at 184.15 146.05 90)
+		(lib_id "Device:R")
+		(at 320.04 118.11 270)
 		(unit 1)
 		(body_style 1)
@@
 		(in_pos_files yes)
 		(dnp no)
-		(fields_autoplaced yes)
-		(property "Reference" "TP2"
-			(at 180.848 140.97 90)
+		(property "Reference" "R23"
+			(at 319.786 115.824 90)
 			(show_name no)
 			(do_not_autoplace no)
@@
 			)
 		)
-		(property "Value" "TestPoint"
-			(at 180.848 143.51 90)
+		(property "Value" "2.2K/1%"
+			(at 318.008 120.396 90)
 			(show_name no)
 			(do_not_autoplace no)
@@
 			)
 		)
-		(property "Footprint" ""
-			(at 184.15 140.97 0)
+		(property "Footprint" "A_HDJ_Library:R_0402_1005Metric"
+			(at 320.04 116.332 90)
 			(hide yes)
 			(show_name no)
@@
 		)
 		(property "Datasheet" ""
-			(at 184.15 140.97 0)
+			(at 320.04 118.11 0)
 			(hide yes)
 			(show_name no)
@@
 			)
 		)
-		(property "Description" "test point"
-			(at 184.15 146.05 0)
+		(property "Description" "Resistor"
+			(at 320.04 118.11 0)
 			(hide yes)
 			(show_name no)
@@
 			)
 		)
+		(pin "2"
+		)
 		(pin "1"
 		)
@@
 			(project "LattepndaCourse"
 				(path "/4e04f3a7-ba43-4db9-8bbc-1a27efcf5abf/dc3c01ed-4c1a-4ffc-b57d-00aa66dee251"
-					(reference "TP2")
+					(reference "R23")
 					(unit 1)
 				)
@@
 	)
 	(symbol
-		(lib_id "Device:C_Small")
-		(at 370.84 275.59 180)
+		(lib_id "Connector:TestPoint")
+		(at 184.15 146.05 90)
 		(unit 1)
 		(body_style 1)
@@
 		(in_pos_files yes)
 		(dnp no)
-		(property "Reference" "C23"
-			(at 371.856 273.558 90)
+		(fields_autoplaced yes)
+		(property "Reference" "TP2"
+			(at 180.848 140.97 90)
 			(show_name no)
 			(do_not_autoplace no)
@@
 			)
 		)
-		(property "Value" "1uF/16V"
-			(at 368.046 275.59 90)
+		(property "Value" "TestPoint"
+			(at 180.848 143.51 90)
 			(show_name no)
 			(do_not_autoplace no)
@@
 			)
 		)
-		(property "Footprint" "A_HDJ_Library:C_0402_1005Metric"
-			(at 370.84 275.59 0)
+		(property "Footprint" ""
+			(at 184.15 140.97 0)
 			(hide yes)
 			(show_name no)
@@
 		)
 		(property "Datasheet" ""
-			(at 370.84 275.59 0)
+			(at 184.15 140.97 0)
 			(hide yes)
 			(show_name no)
@@
 			)
 		)
-		(property "Description" "Unpolarized capacitor, small symbol"
-			(at 370.84 275.59 0)
+		(property "Description" "test point"
+			(at 184.15 146.05 0)
 			(hide yes)
 			(show_name no)
@@
 			)
 		)
-		(pin "2"
-		)
 		(pin "1"
 		)
@@
 			(project "LattepndaCourse"
 				(path "/4e04f3a7-ba43-4db9-8bbc-1a27efcf5abf/dc3c01ed-4c1a-4ffc-b57d-00aa66dee251"
-					(reference "C23")
+					(reference "TP2")
 					(unit 1)
 				)
@@
 	)
 	(symbol
-		(lib_id "Device:R")
-		(at 246.38 77.47 90)
+		(lib_id "Device:C_Small")
+		(at 370.84 275.59 180)
 		(unit 1)
 		(body_style 1)
@@
 		(on_board yes)
 		(in_pos_files yes)
-		(dnp yes)
-		(property "Reference" "R10"
-			(at 241.554 76.454 90)
+		(dnp no)
+		(property "Reference" "C23"
+			(at 371.856 273.558 90)
 			(show_name no)
 			(do_not_autoplace no)
@@
 			)
 		)
-		(property "Value" "100K/1%"
-			(at 247.142 79.502 90)
+		(property "Value" "1uF/16V"
+			(at 368.046 275.59 90)
 			(show_name no)
 			(do_not_autoplace no)
@@
 			)
 		)
-		(property "Footprint" "A_HDJ_Library:R_0402_1005Metric"
-			(at 246.38 79.248 90)
+		(property "Footprint" "A_HDJ_Library:C_0402_1005Metric"
+			(at 370.84 275.59 0)
 			(hide yes)
 			(show_name no)
@@
 		)
 		(property "Datasheet" ""
-			(at 246.38 77.47 0)
+			(at 370.84 275.59 0)
 			(hide yes)
 			(show_name no)
@@
 			)
 		)
-		(property "Description" "Resistor"
-			(at 246.38 77.47 0)
+		(property "Description" "Unpolarized capacitor, small symbol"
+			(at 370.84 275.59 0)
 			(hide yes)
 			(show_name no)
@@
 			(project "LattepndaCourse"
 				(path "/4e04f3a7-ba43-4db9-8bbc-1a27efcf5abf/dc3c01ed-4c1a-4ffc-b57d-00aa66dee251"
-					(reference "R10")
+					(reference "C23")
 					(unit 1)
 				)
@@
 	)
 	(symbol
-		(lib_id "power:PWR_FLAG")
-		(at 105.41 140.97 270)
+		(lib_id "Device:R")
+		(at 246.38 77.47 90)
 		(unit 1)
 		(body_style 1)
@@
 		(on_board yes)
 		(in_pos_files yes)
-		(dnp no)
-		(fields_autoplaced yes)
-		(property "Reference" "#FLG04"
-			(at 107.315 140.97 0)
-			(hide yes)
+		(dnp yes)
+		(property "Reference" "R10"
+			(at 241.554 76.454 90)
 			(show_name no)
 			(do_not_autoplace no)
@@
 			)
 		)
-		(property "Value" "PWR_FLAG"
-			(at 109.22 140.9699 90)
+		(property "Value" "100K/1%"
+			(at 247.142 79.502 90)
 			(show_name no)
 			(do_not_autoplace no)
@@
 					(size 1.27 1.27)
 				)
-				(justify left)
 			)
 		)
-		(property "Footprint" ""
-			(at 105.41 140.97 0)
+		(property "Footprint" "A_HDJ_Library:R_0402_1005Metric"
+			(at 246.38 79.248 90)
 			(hide yes)
 			(show_name no)
@@
 		)
 		(property "Datasheet" ""
-			(at 105.41 140.97 0)
+			(at 246.38 77.47 0)
 			(hide yes)
 			(show_name no)
@@
 			)
 		)
-		(property "Description" "Special symbol for telling ERC where power comes from"
-			(at 105.41 140.97 0)
+		(property "Description" "Resistor"
+			(at 246.38 77.47 0)
 			(hide yes)
 			(show_name no)
@@
 			)
 		)
+		(pin "2"
+		)
 		(pin "1"
 		)
@@
 			(project "LattepndaCourse"
 				(path "/4e04f3a7-ba43-4db9-8bbc-1a27efcf5abf/dc3c01ed-4c1a-4ffc-b57d-00aa66dee251"
-					(reference "#FLG04")
+					(reference "R10")
 					(unit 1)
 				)

Commit message: Hierachi needs some work
Changed lines of the file:
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@@
 		)
 	)
-	(global_label "~{PWR_LED}{slash}~{PSON}"
-		(shape input)
-		(at 297.18 200.66 180)
-		(fields_autoplaced yes)
+	(hierarchical_label "~{PWR_SW}"
+		(shape output)
+		(at 287.02 267.97 180)
 		(effects
 			(font
@@
 			(justify right)
 		)
-		(property "Intersheetrefs" "${INTERSHEET_REFS}"
-			(at 279.3177 200.66 0)
-			(hide yes)
-			(show_name no)
-			(do_not_autoplace no)
-			(effects
-				(font
-					(size 1.27 1.27)
-				)
-				(justify right)
-			)
-		)
 	)
-	(global_label "~{PWR_SW}"
+	(hierarchical_label "~{RST_SW}"
 		(shape output)
-		(at 287.02 267.97 180)
-		(fields_autoplaced yes)
+		(at 351.79 267.97 180)
 		(effects
 			(font
@@
 			(justify right)
 		)
-		(property "Intersheetrefs" "${INTERSHEET_REFS}"
-			(at 276.4149 267.97 0)
-			(hide yes)
-			(show_name no)
-			(do_not_autoplace no)
-			(effects
-				(font
-					(size 1.27 1.27)
-				)
-				(justify right)
-			)
-		)
 	)
-	(global_label "SLS_S3"
+	(hierarchical_label "SLS_S3"
 		(shape input)
 		(at 299.72 173.99 90)
-		(fields_autoplaced yes)
 		(effects
 			(font
@@
 			(justify left)
 		)
-		(property "Intersheetrefs" "${INTERSHEET_REFS}"
-			(at 299.72 164.1711 90)
-			(hide yes)
-			(show_name no)
-			(do_not_autoplace no)
-			(effects
-				(font
-					(size 1.27 1.27)
-				)
-				(justify left)
-			)
-		)
 	)
-	(global_label "~{RST_SW}"
-		(shape output)
-		(at 351.79 267.97 180)
-		(fields_autoplaced yes)
+	(hierarchical_label "~{PWR_LED}{slash}~{PSON}"
+		(shape input)
+		(at 297.18 200.66 180)
 		(effects
 			(font
@@
 			(justify right)
 		)
-		(property "Intersheetrefs" "${INTERSHEET_REFS}"
-			(at 341.7292 267.97 0)
-			(hide yes)
-			(show_name no)
-			(do_not_autoplace no)
-			(effects
-				(font
-					(size 1.27 1.27)
-				)
-				(justify right)
-			)
-		)
 	)

Commit message: Started routing
Parts:
- J2: footprint (none) -> A_HDJ_Library:USB_C_Receptacle_G-Switch_GT-USB-7010ASV
- JP1: footprint (none) -> A_HDJ_Library:PinHeader_1x03_P2.54mm_Vertical
- TP2, TP3, TP4, TP5, TP6, TP7, TP8: footprint (none) -> A_HDJ_Library:TestPoint_Pad_D1.5mm
